File: gatedrive.kicad_pcb (KiCad board)
At the start: 2 copper layers, 50.8 x 54.4 mm, 26 parts, among them IC1 HCPL-316J, IC2 IXDD614PI, p1 POWER SUPPLY CONNECTOR., p2 IGBT CONNECTOR., p3 CONTROLLER CONNECTOR.

Commit message: START
Changed lines of the file:
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@@
     (descr "Resistor, Axial,  RM 10mm, 1/3W,")
     (tags "Resistor, Axial, RM 10mm, 1/3W,")
-    (fp_text reference R4 (at -1.524 2.54 90) (layer F.SilkS)
+    (fp_text reference R4 (at 0 2.286 90) (layer F.SilkS)
       (effects (font (size 1 1) (thickness 0.15)))
     )
@@
     (descr "Resistor, Axial, RM 20mm,")
     (tags "Resistor, Axial, RM 20mm,")
-    (fp_text reference R4 (at 8.382 1.778 180) (layer F.SilkS)
+    (fp_text reference R4 (at 0 -3.302 270) (layer F.SilkS)
       (effects (font (size 1 1) (thickness 0.15)))
     )
@@
     (descr "Resistor, Axial, RM 20mm,")
     (tags "Resistor, Axial, RM 20mm,")
-    (fp_text reference R4 (at 8.382 1.778 180) (layer F.SilkS)
+    (fp_text reference R4 (at 0 3.556 270) (layer F.SilkS)
       (effects (font (size 1 1) (thickness 0.15)))
     )
@@
     (descr "Resistor, Axial,  RM 10mm, 1/3W,")
     (tags "Resistor, Axial, RM 10mm, 1/3W,")
-    (fp_text reference R4 (at -1.524 2.032 90) (layer F.SilkS)
-      (effects (font (size 1 1) (thickness 0.15)))
-    )
+    (fp_text reference R4 (at 0 -1.778 270) (layer F.SilkS)
+      (effects (font (size 1 1) (thickness 0.15)))
+    )

Commit message: START
Routing:
- net G: track 98.1 -> 94.1 mm
- net Net-(D2-Pad1): track 26.6 -> 23.7 mm
Other:
- board text added: "note that gate resistors are easily scalabe to different IGBT sizes."
- board text removed: "note that gate resistors are easily scalabe different IGBT sizes."
Changed lines of the file:
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@@
     (links 58)
     (no_connects 0)
-    (area 108.098286 65.592 181.969715 128.938001)
+    (area 106.419714 65.592 183.648286 128.938001)
     (thickness 1.6)
     (drawings 20)
-    (tracks 137)
+    (tracks 136)
     (zones 0)
     (modules 26)
@@
   )
   (setup
-    (last_trace_width 0.25)
+    (last_trace_width 1.27)
     (user_trace_width 0.254)
     (user_trace_width 0.6)
@@
     (descr "Resistor, Axial,  RM 10mm, 1/3W,")
     (tags "Resistor, Axial, RM 10mm, 1/3W,")
-    (fp_text reference R5 (at -3.556 1.778) (layer F.SilkS)
+    (fp_text reference R5 (at 0 2.032) (layer F.SilkS)
       (effects (font (size 1 1) (thickness 0.15)))
     )
@@
     (descr "Resistor, Axial,  RM 10mm, 1/3W,")
     (tags "Resistor, Axial, RM 10mm, 1/3W,")
-    (fp_text reference R5 (at -3.556 1.778) (layer F.SilkS)
+    (fp_text reference R5 (at 0 2.032) (layer F.SilkS)
       (effects (font (size 1 1) (thickness 0.15)))
     )
@@
     )
   )
-  (gr_text "note that gate resistors are easily scalabe different IGBT sizes." (at 145.034 69.342) (layer Eco1.User)
+  (gr_text "note that gate resistors are easily scalabe to different IGBT sizes." (at 145.034 69.342) (layer Eco1.User)
     (effects (font (size 1.5 1.5) (thickness 0.3)))
   )
@@
   (segment (start 146.431 108.204) (end 149.653 104.982) (width 1.27) (layer B.Cu) (net 6) (status 10))
   (segment (start 149.653 104.982) (end 160.782 104.982) (width 1.27) (layer B.Cu) (net 6) (status 20))
+  (segment (start 163.322 80.518) (end 163.322 82.107793) (width 2) (layer B.Cu) (net 8))
+  (segment (start 163.322 82.107793) (end 166.953813 85.739606) (width 2) (layer B.Cu) (net 8))
+  (segment (start 166.953813 85.739606) (end 166.953813 107.060187) (width 2) (layer B.Cu) (net 8))
+  (segment (start 166.953813 107.060187) (end 166.637491 107.376509) (width 2) (layer B.Cu) (net 8))
   (segment (start 163.162 116.078) (end 163.162 110.852) (width 2) (layer B.Cu) (net 8) (status 10))
   (segment (start 163.162 116.078) (end 159.766 116.078) (width 2) (layer B.Cu) (net 8) (status 10))
@@
   (segment (start 158.75 74.582) (end 158.75 77.47) (width 2) (layer B.Cu) (net 8) (status 10))
   (segment (start 158.75 77.47) (end 158.75 80.518) (width 2) (layer B.Cu) (net 8) (status 20))
-  (segment (start 161.798 80.518) (end 158.75 77.47) (width 2) (layer B.Cu) (net 8))
   (segment (start 163.322 80.518) (end 158.75 80.518) (width 2) (layer B.Cu) (net 8) (status 30))
   (segment (start 160.782 109.93093) (end 160.782 109.982) (width 2) (layer B.Cu) (net 8) (status 30))
@@
   (segment (start 166.637491 107.376509) (end 164.032 109.982) (width 2) (layer B.Cu) (net 8))
   (segment (start 163.322 80.518) (end 161.798 80.518) (width 2) (layer B.Cu) (net 8) (status 10))
-  (segment (start 166.637491 89.615401) (end 166.637491 107.376509) (width 2) (layer B.Cu) (net 8))
-  (segment (start 163.322 80.518) (end 163.322 86.29991) (width 2) (layer B.Cu) (net 8) (status 10))
-  (segment (start 163.322 86.29991) (end 166.637491 89.615401) (width 2) (layer B.Cu) (net 8))
   (segment (start 131.875 80.645) (end 128.063499 80.645) (width 0.6) (layer B.Cu) (net 9) (status 10))
   (segment (start 126.412499 82.296) (end 123.952 82.296) (width 0.6) (layer B.Cu) (net 9) (status 20))
@@
   (segment (start 158.75 94.582) (end 160.782 94.582) (width 2) (layer B.Cu) (net 13) (status 10))
   (segment (start 160.782 94.582) (end 164.337481 94.582) (width 2) (layer B.Cu) (net 13) (status 20))
-  (segment (start 158.75 92.55) (end 160.782 94.582) (width 2) (layer B.Cu) (net 13))
   (segment (start 158.75 90.678) (end 158.75 92.55) (width 2) (layer B.Cu) (net 13) (status 10))
   (segment (start 158.75 94.582) (end 158.75 90.678) (width 2) (layer B.Cu) (net 13) (status 30))
