File: gatedrive.kicad_pcb (KiCad board)
At the start: 2 copper layers, 189.9 x 101 mm, 155 parts, among them IC201 HCPL-316J, IC202 IXDD614PI, IC301 HCPL-316J, IC302 IXDD614PI, IC401 HCPL-316J, IC402 IXDD614PI, IC501 HCPL-316J, IC502 IXDD614PI, IC601 HCPL-316J, IC602 IXDD614PI, IC701 HCPL-316J, IC702 IXDD614PI, IC901 HCPL-316J, IC902 IXDD614PI, P101 Mic General Connector, P201 CONN_01X03, P202 CONN_01X03, P301 CONN_01X03, P302 CONN_01X03, P401 CONN_01X03, P402 CONN_01X03, P501 CONN_01X03, P502 CONN_01X03, P601 CONN_01X03, P602 CONN_01X03, P701 CONN_01X03, P702 CONN_01X03, P801 FromShuntResistor, P802 FromNtc, P901 CONN_01X03, P902 CONN_01X03, U802 LM339

Commit message: parting the protection from the GD
Parts:
- removed C1 (x2): 0.1u, gatedrive:C_Disc
- removed the C602 at (125.1, 49.5)
- removed C801: 33pf, gatedrive:C_Disc
- removed C802: 33p, gatedrive:C_Disc
- removed D801: ZENER, Diodes_ThroughHole:Diode_DO-41_SOD81_Horizontal_RM10
- removed P801: FromShuntResistor, Terminal_Blocks:TerminalBlock_Pheonix_MKDS1.5-2pol
- removed P802: FromNtc, Terminal_Blocks:TerminalBlock_Pheonix_MKDS1.5-2pol
- removed R801, R802, R811: 1.24k, Resistors_ThroughHole:Resistor_Horizontal_RM10mm
- removed R803: 20k, Resistors_ThroughHole:Resistor_Horizontal_RM10mm
- removed R804, R805: 61.9k, Resistors_ThroughHole:Resistor_Horizontal_RM10mm
- removed R806: 560, Resistors_ThroughHole:Resistor_Horizontal_RM10mm
- removed R807: 10K, Resistors_ThroughHole:Resistor_Horizontal_RM10mm
- removed R808, R810: 10k, Resistors_ThroughHole:Resistor_Horizontal_RM10mm
- removed R809: 2.2MEG, Resistors_ThroughHole:Resistor_Horizontal_RM10mm
- removed RV801: 10k, Potentiometers:Potentiometer_Bourns_3296W_3-8Zoll_Inline_ScrewUp
- removed U802: LM339, Housings_DIP:DIP-14_W7.62mm_LongPads
- added 2: MountingHole_3.2mm_M3, Mounting_Holes:MountingHole_3.2mm_M3, F.Cu at (102.9, 141.0)
- added 2: MountingHole_3.2mm_M3, Mounting_Holes:MountingHole_3.2mm_M3, F.Cu at (46.4, 50.2)
- added 2: MountingHole_3.2mm_M3, Mounting_Holes:MountingHole_3.2mm_M3, F.Cu at (174.6, 50.2)
- added 2: MountingHole_3.2mm_M3, Mounting_Holes:MountingHole_3.2mm_M3, F.Cu at (173.4, 141.0)
- added 2: MountingHole_3.2mm_M3, Mounting_Holes:MountingHole_3.2mm_M3, F.Cu at (32.4, 141.0)
- added P1: CONN_01X03, Pin_Headers:Pin_Header_Angled_1x04, F.Cu at (188.0, 52.7)
- P101: footprint Socket_Strips:Socket_Strip_Angled_1x12 -> gatedrive:MICCONN
- moved C601 21.7 mm to (89.5, 59.7)
- moved R601 21.7 mm to (96.5, 62.9)
- moved C202 20.5 mm to (188.0, 73.0)
- moved C204 20.4 mm to (177.2, 85.7)
- moved C303 20.4 mm to (161.3, 81.9)
- moved C304 20.4 mm to (153.7, 85.7)
- moved C403 20.4 mm to (137.8, 81.9)
- moved D202 20.4 mm to (187.3, 107.3)
- moved IC202 20.4 mm to (175.3, 92.1)
- moved IC302 20.4 mm to (151.8, 92.1)
- moved P101 20.4 mm to (135.9, 51.4)
- moved P202 20.4 mm to (187.3, 139.7)
- moved R204 20.4 mm to (187.3, 88.3)
- moved R205 20.4 mm to (187.3, 113.7)
- moved R401 20.4 mm to (141.6, 62.9)
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Connections:
- P201 pad 1: COM7 -> 15V7
- P201 pad 2: 15V7 -> COM7
- P301 pad 1: COM6 -> 15V6
- P301 pad 2: 15V6 -> COM6
- P401 pad 1: COM5 -> 15V5
- P401 pad 2: 15V5 -> COM5
- P501 pad 1: COM4 -> 15V4
- P501 pad 2: 15V4 -> COM4
- P601 pad 1: COM3 -> 15V3
- P601 pad 2: 15V3 -> COM3
- P701 pad 1: COM2 -> 15V2
- P701 pad 2: 15V2 -> COM2
- P901 pad 1: COM1 -> 15V1
- P901 pad 2: 15V1 -> COM1
Routing:
- net Net-(C802-Pad1): track 42.4 -> 0.00 mm
- net Net-(D801-Pad1): track 33.7 -> 0.00 mm
- net Net-(P802-Pad2): track 32.1 -> 0.00 mm
- net /protection/+ve: track 32.1 -> 0.00 mm
- net ~OVERTEMP: track 90.9 -> 59.8 mm
- net /protection/-ve: track 27.5 -> 0.00 mm
- net ~FAULT: track 324.0 -> 298.9 mm
- net Net-(C801-Pad1): track 22.8 -> 0.00 mm
- net Net-(R808-Pad2): track 17.5 -> 0.00 mm
- net +5V: track 96.4 -> 80.6 mm
- net Net-(D801-Pad2): track 11.4 -> 0.00 mm
- net Net-(RV801-Pad2): track 9.04 -> 0.00 mm
- net Net-(P801-Pad1): track 6.96 -> 0.00 mm
- net ~RST: track 192.5 -> 189.8 mm
- net 15V1: track 8.12 -> 9.53 mm
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Other:
- board size 189.9 x 101 mm -> 166.4 x 101.6 mm
- board text added: "+5v"
- board text added: "2016"
- board text added: "Anas Ahmad"
- board text added: "COLLECTOR"
- board text added: "EMITTER (COM)"
- board text added: "GATE"
- board text added: "GateDriver"
- board text added: "T1.."
- board text added: "T2.."
- board text added: "T3.."
- board text added: "T4.."
- board text added: "T5.."
- board text added: "T6.."
- board text added: "T7.."
- board text added: "~FAULT.."
- board text added: "~OVERTEMP"
- board text added: "~RST.."
- board text removed: "LENGTH = 20 cm"
- board text removed: "T1 >"
