File: GD1.sch (KiCad schematic (older format))
At the start: 19 parts, among them IC1 HCPL-316J, IC2 IXDD614PI, P2 CONN_01X03, P3 CONN_01X03

Commit message: uding HCPL-361J modified symbol
Parts:
- IC1: symbol HCPL-316J-RESCUE-gatedrive -> HCPL-316J
Connections:
- wire segments 41 -> 52
Other:
- moved on the sheet: C3, C5, D1, IC2, R2, R3, R4

Commit message: cleaning the schematic
Connections:
- wire segments 52 -> 42
Changed lines of the file:
@@
 a cap to ensure soft turn-off, recommended by datasheet of hcpl.
 Wire Wire Line
-	6850 4950 7000 4950
+	6850 4950 7600 4950
 Wire Wire Line
-	7000 4950 7600 4950
+	5750 4950 6550 4950
 Wire Wire Line
-	5750 4950 6350 4950
+	5750 5050 5750 5150
 Wire Wire Line
-	6350 4950 6550 4950
-Wire Wire Line
-	5750 5050 5750 5100
-Wire Wire Line
-	5750 5100 5750 5150
-Wire Wire Line
-	5750 4750 5750 4800
-Wire Wire Line
-	5750 4800 5750 4850
+	5750 4750 5750 4850
 Connection ~ 6150 4100
 Wire Wire Line
@@
 	6150 4100 6300 4100
 Wire Wire Line
-	6150 4050 6150 4100
-Wire Wire Line
-	6150 4100 6150 4650
+	6150 4050 6150 4650
 Connection ~ 8450 4950
 Wire Wire Line
@@
 Connection ~ 7000 4950
 Wire Wire Line
-	3625 4650 4000 4650
+	3625 4650 4850 4650
 Wire Wire Line
-	4000 4650 4850 4650
-Wire Wire Line
-	8350 4950 8450 4950
-Wire Wire Line
-	8450 4950 8900 4950
-Wire Wire Line
-	8900 4950 9050 4950
+	8350 4950 9050 4950
 Wire Wire Line
 	9350 4950 9450 4950
 Wire Wire Line
-	9750 4950 9950 4950
-Wire Wire Line
-	9950 4950 10200 4950
+	9750 4950 10200 4950
 Wire Wire Line
 	9750 5250 9950 5250
@@
 	5800 4450 5800 4350
 Wire Wire Line
-	5900 5100 5900 5200
-Wire Wire Line
-	5900 5200 5900 5300
+	5900 5100 5900 5300
 Wire Wire Line
 	5900 5100 5750 5100

Commit message: completion of the layout, initial layout of the protection circuit, reducing number of circuit to 7
Parts:
- C1, C2, C3, C5, C6, C7: footprint Capacitors_ThroughHole:C_Disc_D3_P2.5 -> gatedrive:C_Disc; symbol CP1 -> C
- C4: symbol CP1 -> C
- D1: footprint Diodes_ThroughHole:Diode_DO-201AD_Horizontal_RM15 -> Diodes_ThroughHole:Diode_DO-41_SOD81_Horizontal_RM10
- R1: footprint Resistors_ThroughHole:Resistor_Vertical_RM5mm -> Resistors_ThroughHole:Resistor_Horizontal_RM10mm
- R5, R6: footprint Resistors_ThroughHole:Resistor_Horizontal_RM20mm -> gatedrive:Resistor_multi
Changed lines of the file:
@@
 EESchema Schematic File Version 2
+LIBS:Symbols_DCDC-ACDC-Converter_RevC_20Jul2012
+LIBS:Symbols_EN60617_13Mar2013
+LIBS:Symbols_EN60617-10_HF-Radio_DRAFT_12Sep2013
+LIBS:Symbols_ICs-Diskrete_RevD10
+LIBS:Symbols_ICs-Opto_RevB_16Sep2013
+LIBS:Symbols_Microcontroller_Philips-NXP_RevA_06Oct2013
+LIBS:SymbolsSimilarEN60617+oldDIN617-RevE8
+LIBS:Symbols_Socket-DIN41612_RevA
+LIBS:Symbols_Transformer-Diskrete_RevA
 LIBS:power
 LIBS:device
@@
 F 0 "D1" H 6950 3976 50  0000 C CNN
 F 1 "RGPO2-20" H 6950 3900 50  0000 C CNN
-F 2 "Diodes_ThroughHole:Diode_DO-201AD_Horizontal_RM15" H 6950 4100 50  0001 C CNN
+F 2 "Diodes_ThroughHole:Diode_DO-41_SOD81_Horizontal_RM10" H 6950 4100 50  0001 C CNN
 F 3 "" H 6950 4100 50  0000 C CNN
 F 4 "El-Amir" H 6950 4100 60  0001 C CNN "Supplier"
@@
 F 0 "R1" V 3525 4500 50  0000 C CNN
 F 1 "10K" V 3625 4500 50  0000 C CNN
-F 2 "Resistors_ThroughHole:Resistor_Vertical_RM5mm" V 3555 4500 50  0001 C CNN
+F 2 "Resistors_ThroughHole:Resistor_Horizontal_RM10mm" V 3555 4500 50  0001 C CNN
 F 3 "" H 3625 4500 50  0000 C CNN
 F 4 "EL AMIR" H 3625 4500 60  0001 C CNN "Supplier"
@@
 $EndComp
 $Comp
-L CP1 C1
+L C C1
 U 1 1 56EF13D1
 P 4450 2150
 F 0 "C1" H 4150 2150 50  0000 C CNN
 F 1 "0.1uF" H 4250 2050 50  0000 C CNN
-F 2 "Capacitors_ThroughHole:C_Disc_D3_P2.5" H 4488 2000 50  0001 C CNN
+F 2 "gatedrive:C_Disc" H 4488 2000 50  0001 C CNN
 F 3 "" H 4450 2150 50  0000 C CNN
 F 4 "EL AMIR" H 4450 2150 60  0001 C CNN "Supplier"
@@
 $EndComp
 $Comp
-L CP1 C3
+L C C3
 U 1 1 56EF13D7
 P 6150 3900
-F 0 "C3" H 6600 3900 50  0000 C CNN
+F 0 "C3" H 6650 3900 50  0000 C CNN
 F 1 "100pF" H 6400 3900 50  0000 C CNN
-F 2 "Capacitors_ThroughHole:C_Disc_D3_P2.5" H 6188 3750 50  0001 C CNN
+F 2 "gatedrive:C_Disc" H 6188 3750 50  0001 C CNN
 F 3 "" H 6150 3900 50  0000 C CNN
 	1    6150 3900
@@
 $EndComp
 $Comp
-L CP1 C7
+L C C7
 U 1 1 56EF13E1
 P 8850 2150
 F 0 "C7" H 8450 2150 50  0000 C CNN
 F 1 "0.1uF" H 8450 2050 50  0000 C CNN
-F 2 "Capacitors_ThroughHole:C_Disc_D3_P2.5" H 8888 2000 50  0001 C CNN
+F 2 "gatedrive:C_Disc" H 8888 2000 50  0001 C CNN
 F 3 "" H 8850 2150 50  0000 C CNN
 	1    8850 2150
@@
 $EndComp
 $Comp
-L CP1 C6
+L C C6
 U 1 1 56EF13E7
 P 7750 2150
 F 0 "C6" H 7400 2150 50  0000 C CNN
 F 1 "0.1uF" H 7400 2050 50  0000 C CNN
-F 2 "Capacitors_ThroughHole:C_Disc_D3_P2.5" H 7788 2000 50  0001 C CNN
+F 2 "gatedrive:C_Disc" H 7788 2000 50  0001 C CNN
 F 3 "" H 7750 2150 50  0000 C CNN
 	1    7750 2150
@@
 $EndComp
 $Comp
-L CP1 C2
+L C C2
 U 1 1 56EF13EA
 P 5500 2150
 F 0 "C2" H 5150 2150 50  0000 C CNN
 F 1 "0.1uF" H 5150 2050 50  0000 C CNN
-F 2 "Capacitors_ThroughHole:C_Disc_D3_P2.5" H 5538 2000 50  0001 C CNN
+F 2 "gatedrive:C_Disc" H 5538 2000 50  0001 C CNN
 F 3 "" H 5500 2150 50  0000 C CNN
 	1    5500 2150
@@
 $EndComp
 $Comp
-L CP1 C4
+L C C4
 U 1 1 56EF037D
 P 6600 2150
@@
 Pull-Down resistor recommended by the data sheet\n based on vbe=0.6 which I am not so sure of.
 $Comp
-L CP1 C5
+L C C5
 U 1 1 56EF142B
 P 7000 4600
 F 0 "C5" H 7240 4630 50  0000 C CNN
 F 1 "10nF" H 7250 4550 50  0000 C CNN
-F 2 "Capacitors_ThroughHole:C_Disc_D3_P2.5" H 7038 4450 50  0001 C CNN
+F 2 "gatedrive:C_Disc" H 7038 4450 50  0001 C CNN
 F 3 "" H 7000 4600 50  0000 C CNN
 	1    7000 4600
@@
 F 0 "R5" V 9600 4980 50  0000 C CNN
 F 1 "60" V 9500 4950 50  0000 C CNN
-F 2 "Resistors_ThroughHole:Resistor_Horizontal_RM20mm" V 9530 4950 50  0001 C CNN
+F 2 "gatedrive:Resistor_multi" V 9530 4950 50  0001 C CNN
 F 3 "" H 9600 4950 50  0000 C CNN
 F 4 "Al amir" H 9600 4950 60  0001 C CNN "Supplier"
@@
 F 0 "R6" V 9600 5240 50  0000 C CNN
 F 1 "30ohm ,0.5W" V 9500 5250 50  0000 C CNN
-F 2 "Resistors_ThroughHole:Resistor_Horizontal_RM20mm" V 9530 5250 50  0001 C CNN
+F 2 "gatedrive:Resistor_multi" V 9530 5250 50  0001 C CNN
 F 3 "" H 9600 5250 50  0000 C CNN
 F 4 "Supplier_name" H 9600 5250 60  0001 C CNN "Supplier"
@@
 Text Notes 5300 2850 0    60   ~ 0
 0.1 uF are bypass caps, the 330 pF is the fault filter cap.
-Text Notes 5950 3800 0    39   ~ 0
+Text Notes 5550 3800 0    39   ~ 0
 blanking capacitor
 Text Notes 3525 4650 1    30   ~ 0

Commit message: packup
Parts:
- removed C1, C2, C6, C7: 0.1uF, gatedrive:C_Disc, symbol C
- removed C3: 100pF, gatedrive:C_Disc, symbol C
- removed C4: 330pF, Capacitors_ThroughHole:C_Disc_D3_P2.5, symbol C
- removed C5: 10nF, gatedrive:C_Disc, symbol C
- removed D1: RGPO2-20, Diodes_ThroughHole:Diode_DO-41_SOD81_Horizontal_RM10, symbol D
- removed D2: ~, Diodes_ThroughHole:Diode_DO-201AD_Horizontal_RM15, symbol D
- removed IC1: HCPL-316J, Housings_SOIC:SOIC-16_7.5x10.3mm_Pitch1.27mm, symbol HCPL-316J
- removed IC2: IXDD614PI, gatedrive:DIP-8_W7.62mm_LongPads, symbol IXDD614PI-RESCUE-gatedrive
- removed P2, P3: CONN_01X03, Pin_Headers:Pin_Header_Angled_1x03, symbol CONN_01X03
- removed R1: 10K, Resistors_ThroughHole:Resistor_Horizontal_RM10mm, symbol R
- removed R2: 25K, Resistors_ThroughHole:Resistor_Horizontal_RM10mm, symbol R
- removed R3, R4: 100, Resistors_ThroughHole:Resistor_Horizontal_RM10mm, symbol R
- removed R5: 60, gatedrive:Resistor_multi, symbol R
- removed R6: 30ohm ,0.5W, gatedrive:Resistor_multi, symbol R
- added C901, C903, C904, C905: 0.1uF, gatedrive:C_Disc, symbol C_Small
- added C902: 330pF, gatedrive:C_Disc, symbol C_Small
- added C906: 100pF, gatedrive:C_Disc, symbol C_Small
- added C907: 10nF, gatedrive:C_Disc, symbol C_Small
- added D901: RGPO2-20, Diodes_ThroughHole:Diode_DO-41_SOD81_Horizontal_RM10, symbol D
- added D902: ~, Diodes_ThroughHole:Diode_DO-201AD_Horizontal_RM15, symbol D
- added IC901: HCPL-316J, Housings_SOIC:SOIC-16_7.5x10.3mm_Pitch1.27mm, symbol HCPL-316J
- added IC902: IXDD614PI, gatedrive:DIP-8_W7.62mm_LongPads, symbol IXDD614PI
- added P901, P902: CONN_01X03, gatedrive:conn, symbol CONN_01X03
- added R901: 10K, Resistors_ThroughHole:Resistor_Horizontal_RM10mm, symbol R_Small
- added R902: 25K, Resistors_ThroughHole:Resistor_Horizontal_RM10mm, symbol R_Small
- added R903, R904: 100, Resistors_ThroughHole:Resistor_Horizontal_RM10mm, symbol R_Small
- added R905: 60, gatedrive:Resistor_multi, symbol R_Small
- added R906: 30ohm ,0.5W, gatedrive:Resistor_multi, symbol R_Small
Connections:
- net labels added: +5V, -5v1, 1, 15V1, 4, GND, c1
- net labels removed: -5V1, 15v1, C1, GND1, MICSUPP
- wire segments 42 -> 50
Other:
- note added: "5 volt is the vcc of the microcontroller.\n"
- note added: "GND is the ground of the microcontroller.\n"
- note added: "IN PIN IS LEFT OPEN OR CONNECTED TO THE VCC."
- note added: "a cap to ensure soft turn-off,\n recommended by datasheet of hcpl."
- note removed: "Fault pull-up resistor."
- note removed: "GND1 is the ground of the microcontroller.\n"
- note removed: "I'M USING GLOBAL LABELS INSTEAD OF LOCAL LABELS AS THEY LOOK NEATER, LOL."
- note removed: "LEFT OPEN OR CONNECTED TO THE VCC."
- note removed: "MICSUPP is 5 volt from the vcc of the microcontroller.\n"
- note removed: "a cap to ensure soft turn-off, recommended by datasheet of hcpl."

Commit message: parting the protection from the GD
Connections:
- net 15V1: now also P901.1 (P1); no longer P901.2 (P2)
- net COM1: now also P901.2 (P2); no longer P901.1 (P1)
Changed lines of the file:
@@
 IN PIN IS LEFT OPEN OR CONNECTED TO THE VCC.
 $Comp
-L PWR_FLAG #FLG051
+L PWR_FLAG #FLG29
 U 1 1 56EFD9BA
 P 1300 3800
-F 0 "#FLG051" H 1300 3895 50  0001 C CNN
+F 0 "#FLG29" H 1300 3895 50  0001 C CNN
 F 1 "PWR_FLAG" H 1300 4024 50  0000 C CNN
 F 2 "" H 1300 3800 50  0000 C CNN
@@
 $EndComp
 $Comp
-L PWR_FLAG #FLG052
+L PWR_FLAG #FLG30
 U 1 1 56EFD9BB
 P 1750 3800
-F 0 "#FLG052" H 1750 3895 50  0001 C CNN
+F 0 "#FLG30" H 1750 3895 50  0001 C CNN
 F 1 "PWR_FLAG" H 1750 4024 50  0000 C CNN
 F 2 "" H 1750 3800 50  0000 C CNN
@@
 $EndComp
 $Comp
-L PWR_FLAG #FLG053
+L PWR_FLAG #FLG28
 U 1 1 56EFD9BE
 P 1300 2650
-F 0 "#FLG053" H 1300 2745 50  0001 C CNN
+F 0 "#FLG28" H 1300 2745 50  0001 C CNN
 F 1 "PWR_FLAG" H 1300 2874 50  0000 C CNN
 F 2 "" H 1300 2650 50  0000 C CNN
@@
 $EndComp
 $Comp
-L PWR_FLAG #FLG054
+L PWR_FLAG #FLG27
 U 1 1 56EFD9BF
 P 900 3800
-F 0 "#FLG054" H 900 3895 50  0001 C CNN
+F 0 "#FLG27" H 900 3895 50  0001 C CNN
 F 1 "PWR_FLAG" H 900 4024 50  0000 C CNN
 F 2 "" H 900 3800 50  0000 C CNN
@@
 	-1   0    0    1
 $EndComp
+Text GLabel 1550 4775 2    60   Input ~ 0
+COM1
 Text GLabel 1550 4875 2    60   Input ~ 0
-COM1
-Text GLabel 1550 4775 2    60   Input ~ 0
 15V1
 Text GLabel 1550 5425 2    60   Input ~ 0
@@
 -5v1
 $Comp
-L GND #PWR055
+L GND #PWR31
 U 1 1 575D78A0
 P 3650 4750
-F 0 "#PWR055" H 3650 4500 50  0001 C CNN
+F 0 "#PWR31" H 3650 4500 50  0001 C CNN
 F 1 "GND" H 3655 4577 50  0000 C CNN
 F 2 "" H 3650 4750 50  0000 C CNN
@@
 $EndComp
 $Comp
-L +5V #PWR056
+L +5V #PWR30
 U 1 1 575D7EA1
 P 3650 3650
-F 0 "#PWR056" H 3650 3500 50  0001 C CNN
+F 0 "#PWR30" H 3650 3500 50  0001 C CNN
 F 1 "+5V" H 3665 3823 50  0000 C CNN
 F 2 "" H 3650 3650 50  0000 C CNN
@@
 	5150 4250 5150 4350
 Wire Wire Line
-	5150 3950 5150 4050
-Wire Wire Line
 	6000 3850 5150 3850
 Wire Wire Line
@@
 Wire Wire Line
 	6000 3300 6000 3850
-Connection ~ 7800 4050
 Wire Wire Line
 	7700 4050 8450 4050
@@
 	7700 4150 7800 4150
 Wire Wire Line
-	7800 4150 7800 4050
-Wire Wire Line
 	5150 3650 5725 3650
-Connection ~ 5150 4000
 Wire Wire Line
 	8250 4300 8925 4300
@@
 	4050 3750 4050 4050
 Wire Wire Line
-	4050 4050 4150 4050
-Wire Wire Line
 	3650 3650 3650 3950
 Wire Wire Line
@@
 Connection ~ 3650 4250
 Wire Wire Line
-	4050 3950 4150 3950
-Connection ~ 4050 3950
-Wire Wire Line
 	3650 4550 3650 4750
 Wire Wire Line
@@
 Connection ~ 3650 4650
 Wire Wire Line
-	6550 4225 6550 4150
-Connection ~ 6550 4150
-Wire Wire Line
 	5925 4300 6000 4300
 Wire Wire Line
@@
 	5525 4200 5525 4650
 Connection ~ 5525 4300
-Connection ~ 5250 3650
-Wire Wire Line
-	5250 3700 5250 3650
 Wire Wire Line
 	5250 3900 5250 4300
 Connection ~ 5250 4300
-Connection ~ 5525 3650
 Wire Wire Line
 	5150 4000 6800 4000
@@
 	5925 3650 6000 3650
 Connection ~ 6000 3650
-Wire Wire Line
-	5525 3475 5525 3800
 Wire Wire Line
 	4050 4650 4050 3950
@@
 Wire Wire Line
 	3250 3850 3250 3900
+Wire Wire Line
+	4050 3950 4150 3950
+Connection ~ 4050 3950
+Wire Wire Line
+	4050 4050 4150 4050
+Connection ~ 4050 4050
+Wire Wire Line
+	5250 3700 5250 3650
+Connection ~ 5250 3650
+Wire Wire Line
+	5525 3475 5525 3800
+Connection ~ 5525 3650
+Wire Wire Line
+	5150 3950 5150 4050
+Connection ~ 5150 4000
+Wire Wire Line
+	6550 4225 6550 4150
+Connection ~ 6550 4150
+Wire Wire Line
+	7800 4150 7800 4050
+Connection ~ 7800 4050
 $EndSCHEMATC
