File: GD2.sch (KiCad schematic (older format))
At the start: 19 parts, among them IC15 HCPL-316J, IC16 IXDD614PI, P16 CONN_01X03, P17 CONN_01X03

Commit message: packup
Parts:
- removed C50, C51, C55, C56: 0.1uF, gatedrive:C_Disc, symbol CP1
- removed C52: 100pF, gatedrive:C_Disc, symbol CP1
- removed C53: 330pF, gatedrive:C_Disc, symbol CP1
- removed C54: 10nF, gatedrive:C_Disc, symbol CP1
- removed D15: RGPO2-20, Diodes_ThroughHole:Diode_DO-41_SOD81_Horizontal_RM10, symbol D
- removed D16: ~, Diodes_ThroughHole:Diode_DO-201AD_Horizontal_RM15, symbol D
- removed IC15: HCPL-316J, Housings_SOIC:SOIC-16_7.5x10.3mm_Pitch1.27mm, symbol HCPL-316J
- removed IC16: IXDD614PI, gatedrive:DIP-8_W7.62mm_LongPads, symbol IXDD614PI
- removed P16, P17: CONN_01X03, Pin_Headers:Pin_Header_Angled_1x03, symbol CONN_01X03
- removed R43: 10K, Resistors_ThroughHole:Resistor_Horizontal_RM10mm, symbol R
- removed R44: 25K, Resistors_ThroughHole:Resistor_Horizontal_RM10mm, symbol R
- removed R45, R46: 100, Resistors_ThroughHole:Resistor_Horizontal_RM10mm, symbol R
- removed R47: 60, gatedrive:Resistor_multi, symbol R
- removed R48: 30ohm ,0.5W, gatedrive:Resistor_multi, symbol R
- added C701, C703, C704, C705: 0.1uF, gatedrive:C_Disc, symbol C_Small
- added C702: 330pF, gatedrive:C_Disc, symbol C_Small
- added C706: 100pF, gatedrive:C_Disc, symbol C_Small
- added C707: 10nF, gatedrive:C_Disc, symbol C_Small
- added D701: RGPO2-20, Diodes_ThroughHole:Diode_DO-41_SOD81_Horizontal_RM10, symbol D
- added D702: ~, Diodes_ThroughHole:Diode_DO-201AD_Horizontal_RM15, symbol D
- added IC701: HCPL-316J, Housings_SOIC:SOIC-16_7.5x10.3mm_Pitch1.27mm, symbol HCPL-316J
- added IC702: IXDD614PI, gatedrive:DIP-8_W7.62mm_LongPads, symbol IXDD614PI
- added P701, P702: CONN_01X03, gatedrive:conn, symbol CONN_01X03
- added R701: 10K, Resistors_ThroughHole:Resistor_Horizontal_RM10mm, symbol R_Small
- added R702: 25K, Resistors_ThroughHole:Resistor_Horizontal_RM10mm, symbol R_Small
- added R703, R704: 100, Resistors_ThroughHole:Resistor_Horizontal_RM10mm, symbol R_Small
- added R705: 60, gatedrive:Resistor_multi, symbol R_Small
- added R706: 30ohm ,0.5W, gatedrive:Resistor_multi, symbol R_Small
Connections:
- net 15V2: now also C704.2, C705.1, IC701.12 (Vc), IC701.13 (Vcc2), IC702.1 (VCC), IC702.3 (EN), IC702.8 (VCC), P701.2 (P2)
- net COM2: now also C703.2, C704.1, C706.2, IC701.16 (VE), P701.1 (P1), P702.3 (P3)
- net G2: now also P702.1 (P1), R705.2, R706.2
- net T2: now also IC701.1 (Vin+)
- net ~FAULT: now also C702.1, IC701.6 (~FAULT), R701.1
- net ~RST: now also IC701.5 (~RESET)
- new net: IC701.11 (Vout), R702.2, R704.2
- new net: C706.1, IC701.14 (DESAT), R703.1
- new net: C707.1, IC702.2 (IN), R704.1
- new net: D701.2 (A), R703.2
- new net: D702.1 (K), R705.1
- new net: D702.2 (A), IC702.6 (OUT), IC702.7 (OUT), R706.1
- new net +5V: C701.1, IC701.3 (Vcc1), R701.2
- new net -5v2: C703.1, C705.2, C707.2, IC701.10 (VEE), IC701.9 (VEE), IC702.4 (GND), IC702.5 (GND), P701.3 (P3), R702.1
- new net GND: C701.2, C702.2, IC701.2 (Vin-), IC701.4 (GND1), IC701.8 (Vled1-)
- new net c2: D701.1 (K), P702.2 (P2)
Other:
- note added: "5 volt is the vcc of the microcontroller.\n"
- note added: "COM is the auxiliary emitter of the IGBT."
- note added: "GND is the ground of the microcontroller.\n"
- note added: "IN PIN IS LEFT OPEN OR CONNECTED TO THE VCC."
- note added: "a cap to ensure soft turn-off,\n recommended by datasheet of hcpl."
- note removed: "COM2 is the auxiliary emitter of the IGBT."
- note removed: "Fault pull-up resistor."
- note removed: "GND1 is the ground of the microcontroller.\n"
- note removed: "I'M USING GLOBAL LABELS INSTEAD OF LOCAL LABELS AS THEY LOOK NEATER, LOL."
- note removed: "LEFT OPEN OR CONNECTED TO THE VCC."
- note removed: "MICSUPP is 5 volt from the vcc of the microcontroller.\n"
- note removed: "a cap to ensure soft turn-off, recommended by datasheet of hcpl."

Commit message: parting the protection from the GD
Connections:
- net 15V2: now also P701.1 (P1); no longer P701.2 (P2)
- net COM2: now also P701.2 (P2); no longer P701.1 (P1)
Changed lines of the file:
@@
 IN PIN IS LEFT OPEN OR CONNECTED TO THE VCC.
 $Comp
-L PWR_FLAG #FLG039
+L PWR_FLAG #FLG25
 U 1 1 575FED23
 P 1300 3800
-F 0 "#FLG039" H 1300 3895 50  0001 C CNN
+F 0 "#FLG25" H 1300 3895 50  0001 C CNN
 F 1 "PWR_FLAG" H 1300 4024 50  0000 C CNN
 F 2 "" H 1300 3800 50  0000 C CNN
@@
 $EndComp
 $Comp
-L PWR_FLAG #FLG040
+L PWR_FLAG #FLG26
 U 1 1 575FED24
 P 1750 3800
-F 0 "#FLG040" H 1750 3895 50  0001 C CNN
+F 0 "#FLG26" H 1750 3895 50  0001 C CNN
 F 1 "PWR_FLAG" H 1750 4024 50  0000 C CNN
 F 2 "" H 1750 3800 50  0000 C CNN
@@
 $EndComp
 $Comp
-L PWR_FLAG #FLG041
+L PWR_FLAG #FLG24
 U 1 1 575FED27
 P 1300 2650
-F 0 "#FLG041" H 1300 2745 50  0001 C CNN
+F 0 "#FLG24" H 1300 2745 50  0001 C CNN
 F 1 "PWR_FLAG" H 1300 2874 50  0000 C CNN
 F 2 "" H 1300 2650 50  0000 C CNN
@@
 $EndComp
 $Comp
-L PWR_FLAG #FLG042
+L PWR_FLAG #FLG23
 U 1 1 575FED28
 P 900 3800
-F 0 "#FLG042" H 900 3895 50  0001 C CNN
+F 0 "#FLG23" H 900 3895 50  0001 C CNN
 F 1 "PWR_FLAG" H 900 4024 50  0000 C CNN
 F 2 "" H 900 3800 50  0000 C CNN
@@
 	5150 4250 5150 4350
 Wire Wire Line
-	5150 3950 5150 4050
-Wire Wire Line
 	6000 3850 5150 3850
 Wire Wire Line
@@
 Wire Wire Line
 	6000 3300 6000 3850
-Connection ~ 7800 4050
 Wire Wire Line
 	7700 4050 8450 4050
@@
 	7700 4150 7800 4150
 Wire Wire Line
-	7800 4150 7800 4050
-Wire Wire Line
 	5150 3650 5725 3650
-Connection ~ 5150 4000
 Wire Wire Line
 	8250 4300 8925 4300
@@
 	-1   0    0    1
 $EndComp
+Text GLabel 1550 4775 2    60   Input ~ 0
+COM2
 Text GLabel 1550 4875 2    60   Input ~ 0
-COM2
-Text GLabel 1550 4775 2    60   Input ~ 0
 15V2
 Text GLabel 1550 5425 2    60   Input ~ 0
@@
 	3975 4150 4150 4150
 $Comp
-L GND #PWR043
+L GND #PWR22
 U 1 1 575FED31
 P 3650 4750
-F 0 "#PWR043" H 3650 4500 50  0001 C CNN
+F 0 "#PWR22" H 3650 4500 50  0001 C CNN
 F 1 "GND" H 3655 4577 50  0000 C CNN
 F 2 "" H 3650 4750 50  0000 C CNN
@@
 	4050 4050 4150 4050
 $Comp
-L +5V #PWR044
+L +5V #PWR21
 U 1 1 575FED32
 P 3650 3650
-F 0 "#PWR044" H 3650 3500 50  0001 C CNN
+F 0 "#PWR21" H 3650 3500 50  0001 C CNN
 F 1 "+5V" H 3665 3823 50  0000 C CNN
 F 2 "" H 3650 3650 50  0000 C CNN
@@
 Connection ~ 3650 4650
 Wire Wire Line
-	6550 4225 6550 4150
-Connection ~ 6550 4150
-Wire Wire Line
 	3250 3850 3250 3900
 Wire Wire Line
@@
 	5525 4200 5525 4650
 Connection ~ 5525 4300
-Connection ~ 5250 3650
-Wire Wire Line
-	5250 3700 5250 3650
 Wire Wire Line
 	5250 3900 5250 4300
 Connection ~ 5250 4300
-Connection ~ 5525 3650
 $Comp
 L C_Small C704
@@
 Connection ~ 6000 3650
 Wire Wire Line
-	5525 3475 5525 3800
-Wire Wire Line
 	4050 4650 4050 3950
 Text Label 7700 3950 0    60   ~ 0
@@
 Wire Wire Line
 	3250 4100 3250 4650
+Wire Wire Line
+	5250 3700 5250 3650
+Connection ~ 5250 3650
+Wire Wire Line
+	5525 3475 5525 3800
+Connection ~ 5525 3650
+Wire Wire Line
+	5150 3950 5150 4050
+Connection ~ 5150 4000
+Wire Wire Line
+	6550 4225 6550 4150
+Connection ~ 6550 4150
+Wire Wire Line
+	7800 4150 7800 4050
+Connection ~ 7800 4050
 $EndSCHEMATC
