File: GD3.sch (KiCad schematic (older format))
At the start: 19 parts, among them IC13 HCPL-316J, IC14 IXDD614PI, P14 CONN_01X03, P15 CONN_01X03

Commit message: uding HCPL-361J modified symbol
Parts:
- IC13: symbol HCPL-316J-RESCUE-gatedrive -> HCPL-316J
Connections:
- wire segments 43 -> 56
Other:
- moved on the sheet: IC14
Changed lines of the file:
@@
 EESchema Schematic File Version 2
-LIBS:gatedrive-rescue
 LIBS:power
 LIBS:device
@@
 LIBS:contrib
 LIBS:valves
-LIBS:GateDrive
+LIBS:74xgxx
+LIBS:ac-dc
+LIBS:actel
+LIBS:Altera
+LIBS:analog_devices
+LIBS:brooktre
+LIBS:cmos_ieee
+LIBS:dc-dc
+LIBS:diode
+LIBS:elec-unifil
+LIBS:ESD_Protection
+LIBS:ftdi
+LIBS:gennum
+LIBS:graphic
+LIBS:hc11
+LIBS:ir
+LIBS:Lattice
+LIBS:logo
+LIBS:maxim
+LIBS:microchip_dspic33dsc
+LIBS:microchip_pic10mcu
+LIBS:microchip_pic12mcu
+LIBS:microchip_pic16mcu
+LIBS:microchip_pic18mcu
+LIBS:microchip_pic32mcu
+LIBS:motor_drivers
+LIBS:msp430
+LIBS:nordicsemi
+LIBS:nxp_armmcu
+LIBS:onsemi
+LIBS:Oscillators
+LIBS:powerint
+LIBS:Power_Management
+LIBS:pspice
+LIBS:references
+LIBS:relays
+LIBS:rfcom
+LIBS:sensors
+LIBS:silabs
+LIBS:stm8
+LIBS:stm32
+LIBS:supertex
+LIBS:switches
+LIBS:transf
+LIBS:ttl_ieee
+LIBS:video
+LIBS:Worldsemi
+LIBS:Xicor
+LIBS:Zilog
 LIBS:gatedrive-cache
 EELAYER 25 0
@@
 L IXDD614PI-RESCUE-gatedrive IC14
 U 1 1 56EF1F7C
-P 7900 5100
-F 0 "IC14" H 7900 4900 60  0000 C CNN
-F 1 "IXDD614PI" H 7950 5450 60  0000 C CNN
-F 2 "gatedrive:DIP-8_W7.62mm_LongPads" H 7900 5200 60  0001 C CNN
-F 3 "" H 7900 5200 60  0000 C CNN
-F 4 "CHINA[already bought]" H 7900 5100 60  0001 C CNN "Supplier"
-	1    7900 5100
-	1    0    0    -1
-$EndComp
-$Comp
-L HCPL-316J-RESCUE-gatedrive IC13
+P 7950 5100
+AR Path="/56EF1F7C" Ref="IC14"  Part="1"
+AR Path="/56EF055E/56EF1F7C" Ref="IC14"  Part="1"
+F 0 "IC14" H 7950 4900 60  0000 C CNN
+F 1 "IXDD614PI" H 8000 5450 60  0000 C CNN
+F 2 "gatedrive:DIP-8_W7.62mm_LongPads" H 7950 5200 60  0001 C CNN
+F 3 "" H 7950 5200 60  0000 C CNN
+F 4 "CHINA[already bought]" H 7950 5100 60  0001 C CNN "Supplier"
+	1    7950 5100
+	1    0    0    -1
+$EndComp
+$Comp
+L HCPL-316J IC13
 U 1 1 56EF1F7D
-P 5550 4750
-F 0 "IC13" H 5550 4150 60  0000 C CNN
-F 1 "HCPL-316J" H 5300 5200 60  0000 C CNN
-F 2 "Housings_SOIC:SOIC-16_7.5x10.3mm_Pitch1.27mm" H 5550 4750 60  0001 C CNN
-F 3 "" H 5550 4750 60  0000 C CNN
-F 4 "CHINA [ already bought]" H 5550 4750 60  0001 C CNN "Supplier"
-	1    5550 4750
+P 5700 4850
+F 0 "IC13" H 5450 4450 60  0000 C CNN
+F 1 "HCPL-316J" H 5450 5350 60  0000 C CNN
+F 2 "Housings_SOIC:SOIC-16_7.5x10.3mm_Pitch1.27mm" H 5700 4850 60  0001 C CNN
+F 3 "" H 5700 4850 60  0000 C CNN
+F 4 "CHINA [ already bought]" H 5700 4850 60  0001 C CNN "Supplier"
+	1    5700 4850
 	1    0    0    -1
 $EndComp
@@
 a cap to ensure soft turn-off, reCOM3mended by datasheet of hcpl.
 Wire Wire Line
-	6950 4950 7500 4950
-Wire Wire Line
-	6250 4950 6650 4950
-Wire Wire Line
-	6250 5050 6250 5150
-Wire Wire Line
-	6250 4750 6250 4850
+	6950 4950 7150 4950
+Wire Wire Line
+	7150 4950 7550 4950
+Wire Wire Line
+	5900 4950 6500 4950
+Wire Wire Line
+	6500 4950 6650 4950
+Wire Wire Line
+	6250 5050 6250 5100
+Wire Wire Line
+	6250 5100 6250 5150
+Wire Wire Line
+	6250 4750 6250 4800
+Wire Wire Line
+	6250 4800 6250 4850
 Connection ~ 6550 4100
 Wire Wire Line
-	6550 4650 6250 4650
+	5900 4650 6550 4650
 Wire Wire Line
 	6550 4100 6650 4100
 Wire Wire Line
-	6550 4050 6550 4650
+	6550 4650 6550 4100
+Wire Wire Line
+	6550 4100 6550 4050
 Connection ~ 8450 4950
 Wire Wire Line
@@
 Connection ~ 7150 4950
 Wire Wire Line
-	3625 4650 4850 4650
-Wire Wire Line
-	8350 4950 9050 4950
+	3625 4650 4000 4650
+Wire Wire Line
+	4000 4650 5000 4650
+Wire Wire Line
+	8300 4950 8450 4950
+Wire Wire Line
+	8450 4950 8900 4950
+Wire Wire Line
+	8900 4950 9050 4950
 Wire Wire Line
 	9350 4950 9450 4950
 Wire Wire Line
-	9750 4950 10200 4950
+	9750 4950 9950 4950
+Wire Wire Line
+	9950 4950 10200 4950
 Wire Wire Line
 	9750 5250 9950 5250
@@
 Connection ~ 9950 4950
 Wire Wire Line
-	8350 5050 8450 5050
+	8300 5050 8450 5050
 Wire Wire Line
 	8450 5050 8450 4950
@@
 	4400 4350 4400 4550
 Wire Wire Line
-	4400 4550 4850 4550
+	4400 4550 5000 4550
 Wire Wire Line
 	4000 4350 4000 4650
@@
 	4000 5300 4000 4750
 Wire Wire Line
-	4000 4750 4850 4750
-Wire Wire Line
-	4850 5150 4750 5150
+	4000 4750 5000 4750
+Wire Wire Line
+	5000 5150 4750 5150
 Wire Wire Line
 	4750 5150 4750 5300
 Wire Wire Line
-	4850 4850 4400 4850
+	5000 4850 4400 4850
 Wire Wire Line
 	4400 4850 4400 5300
 Wire Wire Line
-	6250 4450 6300 4450
+	5900 4450 6300 4450
 Wire Wire Line
 	6300 4450 6300 4350
@@
 	6500 5000 6500 4950
 Wire Wire Line
-	7500 5050 7175 5050
+	7550 5050 7175 5050
 Wire Wire Line
 	7175 5050 7175 5075
 Text HLabel 900  3800 3    60   Input ~ 0
 T3
-Text HLabel 4850 4450 0    60   Input ~ 0
+Text HLabel 5000 4450 0    60   Input ~ 0
 T3
 Text GLabel 4000 5300 3    60   Input ~ 0
@@
 Text GLabel 4400 5300 3    60   Input ~ 0
 ~RST
-Text GLabel 4850 4950 0    60   Input ~ 0
+Text GLabel 5000 4950 0    60   Input ~ 0
 ~FAULT
 Text GLabel 3625 4350 1    60   Input ~ 0
@@
 	7350 5200 7350 5150
 Wire Wire Line
-	7350 5150 7500 5150
+	7350 5150 7550 5150
 $Comp
 L CONN_01X03 P14
@@
 Text GLabel 7350 5200 3    60   Input ~ 0
 -5V3
-Text GLabel 7500 4850 0    60   Input ~ 0
-15V3
-Text GLabel 8350 4850 2    60   Input ~ 0
-15V3
-Text GLabel 8350 5150 2    60   Input ~ 0
+Text GLabel 7550 4850 0    60   Input ~ 0
+15V3
+Text GLabel 8300 4850 2    60   Input ~ 0
+15V3
+Text GLabel 8300 5150 2    60   Input ~ 0
 -5V3
 Text GLabel 10200 4950 2    60   Input ~ 0
@@
 Text GLabel 1350 5400 2    60   Input ~ 0
 G3
+Wire Wire Line
+	6250 4750 5900 4750
+Wire Wire Line
+	6250 4850 5900 4850
+Wire Wire Line
+	6250 5050 5900 5050
+Wire Wire Line
+	6250 5150 5900 5150
 $EndSCHEMATC

Commit message: cleaning the schematic
Connections:
- wire segments 56 -> 47
Changed lines of the file:
@@
 a cap to ensure soft turn-off, reCOM3mended by datasheet of hcpl.
 Wire Wire Line
-	6950 4950 7150 4950
+	6950 4950 7550 4950
 Wire Wire Line
-	7150 4950 7550 4950
+	5900 4950 6650 4950
 Wire Wire Line
-	5900 4950 6500 4950
+	6250 5050 6250 5150
 Wire Wire Line
-	6500 4950 6650 4950
-Wire Wire Line
-	6250 5050 6250 5100
-Wire Wire Line
-	6250 5100 6250 5150
-Wire Wire Line
-	6250 4750 6250 4800
-Wire Wire Line
-	6250 4800 6250 4850
+	6250 4750 6250 4850
 Connection ~ 6550 4100
 Wire Wire Line
-	5900 4650 6550 4650
+	6550 4650 5900 4650
 Wire Wire Line
 	6550 4100 6650 4100
 Wire Wire Line
-	6550 4650 6550 4100
-Wire Wire Line
-	6550 4100 6550 4050
+	6550 4050 6550 4650
 Connection ~ 8450 4950
 Wire Wire Line
@@
 Connection ~ 7150 4950
 Wire Wire Line
-	3625 4650 4000 4650
+	3625 4650 5000 4650
 Wire Wire Line
-	4000 4650 5000 4650
-Wire Wire Line
-	8300 4950 8450 4950
-Wire Wire Line
-	8450 4950 8900 4950
-Wire Wire Line
-	8900 4950 9050 4950
+	8300 4950 9050 4950
 Wire Wire Line
 	9350 4950 9450 4950
 Wire Wire Line
-	9750 4950 9950 4950
-Wire Wire Line
-	9950 4950 10200 4950
+	9750 4950 10200 4950
 Wire Wire Line
 	9750 5250 9950 5250

Commit message: completion of the layout, initial layout of the protection circuit, reducing number of circuit to 7
Parts:
- C43, C44, C45, C47, C48, C49: footprint Capacitors_ThroughHole:C_Disc_D3_P2.5 -> gatedrive:C_Disc
- D13: footprint Diodes_ThroughHole:Diode_DO-201AD_Horizontal_RM15 -> Diodes_ThroughHole:Diode_DO-41_SOD81_Horizontal_RM10
- R37: footprint Resistors_ThroughHole:Resistor_Vertical_RM5mm -> Resistors_ThroughHole:Resistor_Horizontal_RM10mm
- R41, R42: footprint Resistors_ThroughHole:Resistor_Horizontal_RM20mm -> gatedrive:Resistor_multi
Changed lines of the file:
@@
 EESchema Schematic File Version 2
+LIBS:Symbols_DCDC-ACDC-Converter_RevC_20Jul2012
+LIBS:Symbols_EN60617_13Mar2013
+LIBS:Symbols_EN60617-10_HF-Radio_DRAFT_12Sep2013
+LIBS:Symbols_ICs-Diskrete_RevD10
+LIBS:Symbols_ICs-Opto_RevB_16Sep2013
+LIBS:Symbols_Microcontroller_Philips-NXP_RevA_06Oct2013
+LIBS:SymbolsSimilarEN60617+oldDIN617-RevE8
+LIBS:Symbols_Socket-DIN41612_RevA
+LIBS:Symbols_Transformer-Diskrete_RevA
 LIBS:power
 LIBS:device
@@
 $Descr A4 11693 8268
 encoding utf-8
-Sheet 8 10
+Sheet 8 9
 Title "IGBT GATE DRIVE SCHEMATIC."
 Date "2016-03-02"
@@
 F 0 "D13" H 7150 3976 50  0000 C CNN
 F 1 "RGPO2-20" H 7150 3900 50  0000 C CNN
-F 2 "Diodes_ThroughHole:Diode_DO-201AD_Horizontal_RM15" H 7150 4100 50  0001 C CNN
+F 2 "Diodes_ThroughHole:Diode_DO-41_SOD81_Horizontal_RM10" H 7150 4100 50  0001 C CNN
 F 3 "" H 7150 4100 50  0000 C CNN
 F 4 "El-Amir" H 7150 4100 60  0001 C CNN "Supplier"
@@
 F 0 "R37" V 3525 4500 50  0000 C CNN
 F 1 "10K" V 3625 4500 50  0000 C CNN
-F 2 "Resistors_ThroughHole:Resistor_Vertical_RM5mm" V 3555 4500 50  0001 C CNN
+F 2 "Resistors_ThroughHole:Resistor_Horizontal_RM10mm" V 3555 4500 50  0001 C CNN
 F 3 "" H 3625 4500 50  0000 C CNN
 F 4 "EL AMIR" H 3625 4500 60  0001 C CNN "Supplier"
@@
 F 0 "C43" H 4150 2150 50  0000 C CNN
 F 1 "0.1uF" H 4250 2050 50  0000 C CNN
-F 2 "Capacitors_ThroughHole:C_Disc_D3_P2.5" H 4488 2000 50  0001 C CNN
+F 2 "gatedrive:C_Disc" H 4488 2000 50  0001 C CNN
 F 3 "" H 4450 2150 50  0000 C CNN
 F 4 "EL AMIR" H 4450 2150 60  0001 C CNN "Supplier"
@@
 F 0 "C45" H 7000 3900 50  0000 C CNN
 F 1 "100pF" H 6800 3900 50  0000 C CNN
-F 2 "Capacitors_ThroughHole:C_Disc_D3_P2.5" H 6588 3750 50  0001 C CNN
+F 2 "gatedrive:C_Disc" H 6588 3750 50  0001 C CNN
 F 3 "" H 6550 3900 50  0000 C CNN
 	1    6550 3900
@@
 F 0 "C49" H 8450 2150 50  0000 C CNN
 F 1 "0.1uF" H 8450 2050 50  0000 C CNN
-F 2 "Capacitors_ThroughHole:C_Disc_D3_P2.5" H 8888 2000 50  0001 C CNN
+F 2 "gatedrive:C_Disc" H 8888 2000 50  0001 C CNN
 F 3 "" H 8850 2150 50  0000 C CNN
 	1    8850 2150
@@
 F 0 "C48" H 7400 2150 50  0000 C CNN
 F 1 "0.1uF" H 7400 2050 50  0000 C CNN
-F 2 "Capacitors_ThroughHole:C_Disc_D3_P2.5" H 7788 2000 50  0001 C CNN
+F 2 "gatedrive:C_Disc" H 7788 2000 50  0001 C CNN
 F 3 "" H 7750 2150 50  0000 C CNN
 	1    7750 2150
@@
 F 0 "C44" H 5150 2150 50  0000 C CNN
 F 1 "0.1uF" H 5150 2050 50  0000 C CNN
-F 2 "Capacitors_ThroughHole:C_Disc_D3_P2.5" H 5538 2000 50  0001 C CNN
+F 2 "gatedrive:C_Disc" H 5538 2000 50  0001 C CNN
 F 3 "" H 5500 2150 50  0000 C CNN
 	1    5500 2150
@@
 LEFT OPEN OR CONNECTED TO THE VCC.
 $Comp
-L PWR_FLAG #FLG043
+L PWR_FLAG #FLG029
 U 1 1 56EF1F8A
 P 1300 3800
-F 0 "#FLG043" H 1300 3895 50  0001 C CNN
+F 0 "#FLG029" H 1300 3895 50  0001 C CNN
 F 1 "PWR_FLAG" H 1300 4024 50  0000 C CNN
 F 2 "" H 1300 3800 50  0000 C CNN
@@
 $EndComp
 $Comp
-L PWR_FLAG #FLG044
+L PWR_FLAG #FLG030
 U 1 1 56EF1F8B
 P 1750 3800
-F 0 "#FLG044" H 1750 3895 50  0001 C CNN
+F 0 "#FLG030" H 1750 3895 50  0001 C CNN
 F 1 "PWR_FLAG" H 1750 4024 50  0000 C CNN
 F 2 "" H 1750 3800 50  0000 C CNN
@@
 $EndComp
 $Comp
-L PWR_FLAG #FLG045
+L PWR_FLAG #FLG031
 U 1 1 56EF1F8C
 P 1750 2650
-F 0 "#FLG045" H 1750 2745 50  0001 C CNN
+F 0 "#FLG031" H 1750 2745 50  0001 C CNN
 F 1 "PWR_FLAG" H 1750 2874 50  0000 C CNN
 F 2 "" H 1750 2650 50  0000 C CNN
@@
 $EndComp
 $Comp
-L PWR_FLAG #FLG046
+L PWR_FLAG #FLG032
 U 1 1 56EF1F8D
 P 900 2650
-F 0 "#FLG046" H 900 2745 50  0001 C CNN
+F 0 "#FLG032" H 900 2745 50  0001 C CNN
 F 1 "PWR_FLAG" H 900 2874 50  0000 C CNN
 F 2 "" H 900 2650 50  0000 C CNN
@@
 $EndComp
 $Comp
-L PWR_FLAG #FLG047
+L PWR_FLAG #FLG033
 U 1 1 56EF1F8E
 P 1300 2650
-F 0 "#FLG047" H 1300 2745 50  0001 C CNN
+F 0 "#FLG033" H 1300 2745 50  0001 C CNN
 F 1 "PWR_FLAG" H 1300 2874 50  0000 C CNN
 F 2 "" H 1300 2650 50  0000 C CNN
@@
 $EndComp
 $Comp
-L PWR_FLAG #FLG048
+L PWR_FLAG #FLG034
 U 1 1 56EF1F8F
 P 900 3800
-F 0 "#FLG048" H 900 3895 50  0001 C CNN
+F 0 "#FLG034" H 900 3895 50  0001 C CNN
 F 1 "PWR_FLAG" H 900 4024 50  0000 C CNN
 F 2 "" H 900 3800 50  0000 C CNN
@@
 F 0 "C47" H 7390 4630 50  0000 C CNN
 F 1 "10nF" H 7400 4550 50  0000 C CNN
-F 2 "Capacitors_ThroughHole:C_Disc_D3_P2.5" H 7188 4450 50  0001 C CNN
+F 2 "gatedrive:C_Disc" H 7188 4450 50  0001 C CNN
 F 3 "" H 7150 4600 50  0000 C CNN
 	1    7150 4600
@@
 F 0 "R41" V 9600 4980 50  0000 C CNN
 F 1 "60" V 9500 4950 50  0000 C CNN
-F 2 "Resistors_ThroughHole:Resistor_Horizontal_RM20mm" V 9530 4950 50  0001 C CNN
+F 2 "gatedrive:Resistor_multi" V 9530 4950 50  0001 C CNN
 F 3 "" H 9600 4950 50  0000 C CNN
 F 4 "Al amir" H 9600 4950 60  0001 C CNN "Supplier"
@@
 F 0 "R42" V 9600 5240 50  0000 C CNN
 F 1 "30ohm ,0.5W" V 9500 5250 50  0000 C CNN
-F 2 "Resistors_ThroughHole:Resistor_Horizontal_RM20mm" V 9530 5250 50  0001 C CNN
+F 2 "gatedrive:Resistor_multi" V 9530 5250 50  0001 C CNN
 F 3 "" H 9600 5250 50  0000 C CNN
 F 4 "Supplier_name" H 9600 5250 60  0001 C CNN "Supplier"
@@
 	6950 4100 7000 4100
 $Comp
-L PWR_FLAG #FLG049
+L PWR_FLAG #FLG035
 U 1 1 56EF1F96
 P 1475 3050
-F 0 "#FLG049" H 1475 3145 50  0001 C CNN
+F 0 "#FLG035" H 1475 3145 50  0001 C CNN
 F 1 "PWR_FLAG" V 1625 3050 50  0000 C CNN
 F 2 "" H 1475 3050 50  0000 C CNN

Commit message: yet another enhancements .
the protection section still is incomplete.
Parts:
- IC14: symbol IXDD614PI-RESCUE-gatedrive -> IXDD614PI
Connections:
- wire segments 47 -> 56
Other:
- moved on the sheet: IC13
Changed lines of the file:
@@
 $Descr A4 11693 8268
 encoding utf-8
-Sheet 8 9
+Sheet 6 9
 Title "IGBT GATE DRIVE SCHEMATIC."
 Date "2016-03-02"
@@
 $EndDescr
 $Comp
-L IXDD614PI-RESCUE-gatedrive IC14
+L IXDD614PI IC14
 U 1 1 56EF1F7C
-P 7950 5100
+P 7900 4950
 AR Path="/56EF1F7C" Ref="IC14"  Part="1"
 AR Path="/56EF055E/56EF1F7C" Ref="IC14"  Part="1"
-F 0 "IC14" H 7950 4900 60  0000 C CNN
-F 1 "IXDD614PI" H 8000 5450 60  0000 C CNN
-F 2 "gatedrive:DIP-8_W7.62mm_LongPads" H 7950 5200 60  0001 C CNN
-F 3 "" H 7950 5200 60  0000 C CNN
-F 4 "CHINA[already bought]" H 7950 5100 60  0001 C CNN "Supplier"
-	1    7950 5100
+F 0 "IC14" H 7900 4600 60  0000 C CNN
+F 1 "IXDD614PI" H 7900 5200 60  0000 C CNN
+F 2 "gatedrive:DIP-8_W7.62mm_LongPads" H 7900 5050 60  0001 C CNN
+F 3 "" H 7900 5050 60  0000 C CNN
+F 4 "CHINA[already bought]" H 7900 4950 60  0001 C CNN "Supplier"
+	1    7900 4950
 	1    0    0    -1
 $EndComp
@@
 L HCPL-316J IC13
 U 1 1 56EF1F7D
-P 5700 4850
-F 0 "IC13" H 5450 4450 60  0000 C CNN
-F 1 "HCPL-316J" H 5450 5350 60  0000 C CNN
-F 2 "Housings_SOIC:SOIC-16_7.5x10.3mm_Pitch1.27mm" H 5700 4850 60  0001 C CNN
-F 3 "" H 5700 4850 60  0000 C CNN
-F 4 "CHINA [ already bought]" H 5700 4850 60  0001 C CNN "Supplier"
-	1    5700 4850
+P 5400 4750
+AR Path="/56EF1F7D" Ref="IC13"  Part="1"
+AR Path="/56EF055E/56EF1F7D" Ref="IC13"  Part="1"
+F 0 "IC13" H 5150 4350 60  0000 C CNN
+F 1 "HCPL-316J" H 5150 5250 60  0000 C CNN
+F 2 "Housings_SOIC:SOIC-16_7.5x10.3mm_Pitch1.27mm" H 5400 4750 60  0001 C CNN
+F 3 "" H 5400 4750 60  0000 C CNN
+F 4 "CHINA [ already bought]" H 5400 4750 60  0001 C CNN "Supplier"
+	1    5400 4750
 	1    0    0    -1
 $EndComp
@@
 a cap to ensure soft turn-off, reCOM3mended by datasheet of hcpl.
 Wire Wire Line
-	6950 4950 7550 4950
-Wire Wire Line
-	5900 4950 6650 4950
-Wire Wire Line
-	6250 5050 6250 5150
-Wire Wire Line
-	6250 4750 6250 4850
+	6950 4950 7150 4950
+Wire Wire Line
+	7150 4950 7500 4950
+Wire Wire Line
+	5900 4950 6500 4950
+Wire Wire Line
+	6500 4950 6650 4950
+Wire Wire Line
+	6250 5050 6250 5100
+Wire Wire Line
+	6250 5100 6250 5150
+Wire Wire Line
+	6250 4750 6250 4800
+Wire Wire Line
+	6250 4800 6250 4850
 Connection ~ 6550 4100
 Wire Wire Line
@@
 	6550 4100 6650 4100
 Wire Wire Line
-	6550 4050 6550 4650
+	6550 4050 6550 4100
+Wire Wire Line
+	6550 4100 6550 4650
 Connection ~ 8450 4950
 Wire Wire Line
@@
 Connection ~ 7150 4950
 Wire Wire Line
-	3625 4650 5000 4650
-Wire Wire Line
-	8300 4950 9050 4950
+	3625 4650 4000 4650
+Wire Wire Line
+	4000 4650 4900 4650
+Wire Wire Line
+	8300 4950 8450 4950
+Wire Wire Line
+	8450 4950 8900 4950
+Wire Wire Line
+	8900 4950 9050 4950
 Wire Wire Line
 	9350 4950 9450 4950
 Wire Wire Line
-	9750 4950 10200 4950
+	9750 4950 9950 4950
+Wire Wire Line
+	9950 4950 10200 4950
 Wire Wire Line
 	9750 5250 9950 5250
@@
 	4400 4350 4400 4550
 Wire Wire Line
-	4400 4550 5000 4550
+	4400 4550 4900 4550
 Wire Wire Line
 	4000 4350 4000 4650
@@
 	4000 5300 4000 4750
 Wire Wire Line
-	4000 4750 5000 4750
-Wire Wire Line
-	5000 5150 4750 5150
+	4000 4750 4900 4750
+Wire Wire Line
+	4900 5150 4750 5150
 Wire Wire Line
 	4750 5150 4750 5300
 Wire Wire Line
-	5000 4850 4400 4850
+	4900 4850 4400 4850
 Wire Wire Line
 	4400 4850 4400 5300
@@
 	6500 5000 6500 4950
 Wire Wire Line
-	7550 5050 7175 5050
+	7500 5050 7175 5050
 Wire Wire Line
 	7175 5050 7175 5075
 Text HLabel 900  3800 3    60   Input ~ 0
 T3
-Text HLabel 5000 4450 0    60   Input ~ 0
+Text HLabel 4900 4450 0    60   Input ~ 0
 T3
 Text GLabel 4000 5300 3    60   Input ~ 0
@@
 Text GLabel 4400 5300 3    60   Input ~ 0
 ~RST
-Text GLabel 5000 4950 0    60   Input ~ 0
+Text GLabel 4900 4950 0    60   Input ~ 0
 ~FAULT
 Text GLabel 3625 4350 1    60   Input ~ 0
@@
 	7350 5200 7350 5150
 Wire Wire Line
-	7350 5150 7550 5150
+	7350 5150 7500 5150
 $Comp
 L CONN_01X03 P14
@@
 Text GLabel 7350 5200 3    60   Input ~ 0
 -5V3
-Text GLabel 7550 4850 0    60   Input ~ 0
+Text GLabel 7500 4850 0    60   Input ~ 0
 15V3
 Text GLabel 8300 4850 2    60   Input ~ 0

Commit message: packup
Parts:
- removed C43, C44, C48, C49: 0.1uF, gatedrive:C_Disc, symbol CP1
- removed C45: 100pF, gatedrive:C_Disc, symbol CP1
- removed C46: 330pF, Capacitors_ThroughHole:C_Disc_D3_P2.5, symbol CP1
- removed C47: 10nF, gatedrive:C_Disc, symbol CP1
- removed D13: RGPO2-20, Diodes_ThroughHole:Diode_DO-41_SOD81_Horizontal_RM10, symbol D
- removed D14: ~, Diodes_ThroughHole:Diode_DO-201AD_Horizontal_RM15, symbol D
- removed IC13: HCPL-316J, Housings_SOIC:SOIC-16_7.5x10.3mm_Pitch1.27mm, symbol HCPL-316J
- removed IC14: IXDD614PI, gatedrive:DIP-8_W7.62mm_LongPads, symbol IXDD614PI
- removed P14, P15: CONN_01X03, Pin_Headers:Pin_Header_Angled_1x03, symbol CONN_01X03
- removed R37: 10K, Resistors_ThroughHole:Resistor_Horizontal_RM10mm, symbol R
- removed R38: 25K, Resistors_ThroughHole:Resistor_Horizontal_RM10mm, symbol R
- removed R39, R40: 100, Resistors_ThroughHole:Resistor_Horizontal_RM10mm, symbol R
- removed R41: 60, gatedrive:Resistor_multi, symbol R
- removed R42: 30ohm ,0.5W, gatedrive:Resistor_multi, symbol R
- added C601, C603, C604, C605: 0.1uF, gatedrive:C_Disc, symbol C_Small
- added C602: 330pF, gatedrive:C_Disc, symbol C_Small
- added C606: 100pF, gatedrive:C_Disc, symbol C_Small
- added C607: 10nF, gatedrive:C_Disc, symbol C_Small
- added D601: RGPO2-20, Diodes_ThroughHole:Diode_DO-41_SOD81_Horizontal_RM10, symbol D
- added D602: ~, Diodes_ThroughHole:Diode_DO-201AD_Horizontal_RM15, symbol D
- added IC601: HCPL-316J, Housings_SOIC:SOIC-16_7.5x10.3mm_Pitch1.27mm, symbol HCPL-316J
- added IC602: IXDD614PI, gatedrive:DIP-8_W7.62mm_LongPads, symbol IXDD614PI
- added P601, P602: CONN_01X03, gatedrive:conn, symbol CONN_01X03
- added R601: 10K, Resistors_ThroughHole:Resistor_Horizontal_RM10mm, symbol R_Small
- added R602: 25K, Resistors_ThroughHole:Resistor_Horizontal_RM10mm, symbol R_Small
- added R603, R604: 100, Resistors_ThroughHole:Resistor_Horizontal_RM10mm, symbol R_Small
- added R605: 60, gatedrive:Resistor_multi, symbol R_Small
- added R606: 30ohm ,0.5W, gatedrive:Resistor_multi, symbol R_Small
Connections:
- net 15V3: now also C604.2, C605.1, IC601.12 (Vc), IC601.13 (Vcc2), IC602.1 (VCC), IC602.3 (EN), IC602.8 (VCC), P601.2 (P2)
- net COM3: now also C603.2, C604.1, C606.2, IC601.16 (VE), P601.1 (P1), P602.3 (P3)
- net G3: now also P602.1 (P1), R605.2, R606.2
- net T3: now also IC601.1 (Vin+)
- net ~FAULT: now also C602.1, IC601.6 (~FAULT), R601.1
- net ~RST: now also IC601.5 (~RESET)
- new net: IC601.11 (Vout), R602.2, R604.2
- new net: C606.1, IC601.14 (DESAT), R603.1
- new net: C607.1, IC602.2 (IN), R604.1
- new net: D601.2 (A), R603.2
- new net: D602.1 (K), R605.1
- new net: D602.2 (A), IC602.6 (OUT), IC602.7 (OUT), R606.1
- new net +5V: C601.1, IC601.3 (Vcc1), R601.2
- new net -5v3: C603.1, C605.2, C607.2, IC601.10 (VEE), IC601.9 (VEE), IC602.4 (GND), IC602.5 (GND), P601.3 (P3), R602.1
- new net GND: C601.2, C602.2, IC601.2 (Vin-), IC601.4 (GND1), IC601.8 (Vled1-)
- new net c3: D601.1 (K), P602.2 (P2)
Other:
- note added: "5 volt is the vcc of the microcontroller.\n"
- note added: "COM is the auxiliary emitter of the IGBT."
- note added: "GND is the ground of the microcontroller.\n"
- note added: "IN PIN IS LEFT OPEN OR CONNECTED TO THE VCC."
- note added: "Pull-Down resistor recommended by the data sheet\n based on vbe=0.6 which I am not so sure of."
- note added: "a cap to ensure soft turn-off,\n recommended by datasheet of hcpl."
- note removed: "COM3 is the auxiliary emitter of the IGBT."
- note removed: "Fault pull-up resistor."
- note removed: "GND1 is the ground of the microcontroller.\n"
- note removed: "I'M USING GLOBAL LABELS INSTEAD OF LOCAL LABELS AS THEY LOOK NEATER, LOL."
- note removed: "LEFT OPEN OR CONNECTED TO THE VCC."
- note removed: "MICSUPP is 5 volt from the vcc of the microcontroller.\n"
- note removed: "Pull-Down resistor reCOM3mended by the data sheet\n based on vbe=0.6 which I am not so sure of."
- note removed: "a cap to ensure soft turn-off, reCOM3mended by datasheet of hcpl."
