File: GD3.sch (KiCad schematic (older format))
At the start: 19 parts, among them IC601 HCPL-316J, IC602 IXDD614PI, P601 CONN_01X03, P602 CONN_01X03

Commit message: parting the protection from the GD
Connections:
- net 15V3: now also P601.1 (P1); no longer P601.2 (P2)
- net COM3: now also P601.2 (P2); no longer P601.1 (P1)
Changed lines of the file:
@@
 IN PIN IS LEFT OPEN OR CONNECTED TO THE VCC.
 $Comp
-L PWR_FLAG #FLG033
+L PWR_FLAG #FLG21
 U 1 1 575FF0FC
 P 1300 3800
-F 0 "#FLG033" H 1300 3895 50  0001 C CNN
+F 0 "#FLG21" H 1300 3895 50  0001 C CNN
 F 1 "PWR_FLAG" H 1300 4024 50  0000 C CNN
 F 2 "" H 1300 3800 50  0000 C CNN
@@
 $EndComp
 $Comp
-L PWR_FLAG #FLG034
+L PWR_FLAG #FLG22
 U 1 1 575FF0FD
 P 1750 3800
-F 0 "#FLG034" H 1750 3895 50  0001 C CNN
+F 0 "#FLG22" H 1750 3895 50  0001 C CNN
 F 1 "PWR_FLAG" H 1750 4024 50  0000 C CNN
 F 2 "" H 1750 3800 50  0000 C CNN
@@
 $EndComp
 $Comp
-L PWR_FLAG #FLG035
+L PWR_FLAG #FLG20
 U 1 1 575FF100
 P 1300 2650
-F 0 "#FLG035" H 1300 2745 50  0001 C CNN
+F 0 "#FLG20" H 1300 2745 50  0001 C CNN
 F 1 "PWR_FLAG" H 1300 2874 50  0000 C CNN
 F 2 "" H 1300 2650 50  0000 C CNN
@@
 $EndComp
 $Comp
-L PWR_FLAG #FLG036
+L PWR_FLAG #FLG19
 U 1 1 575FF101
 P 900 3800
-F 0 "#FLG036" H 900 3895 50  0001 C CNN
+F 0 "#FLG19" H 900 3895 50  0001 C CNN
 F 1 "PWR_FLAG" H 900 4024 50  0000 C CNN
 F 2 "" H 900 3800 50  0000 C CNN
@@
 	5150 4250 5150 4350
 Wire Wire Line
-	5150 3950 5150 4050
-Wire Wire Line
 	6000 3850 5150 3850
 Wire Wire Line
@@
 Wire Wire Line
 	6000 3300 6000 3850
-Connection ~ 7800 4050
 Wire Wire Line
 	7700 4050 8450 4050
@@
 	7700 4150 7800 4150
 Wire Wire Line
-	7800 4150 7800 4050
-Wire Wire Line
 	5150 3650 5725 3650
-Connection ~ 5150 4000
 Wire Wire Line
 	8250 4300 8925 4300
@@
 	-1   0    0    1
 $EndComp
+Text GLabel 1550 4775 2    60   Input ~ 0
+COM3
 Text GLabel 1550 4875 2    60   Input ~ 0
-COM3
-Text GLabel 1550 4775 2    60   Input ~ 0
 15V3
 Text GLabel 1550 5425 2    60   Input ~ 0
@@
 	3975 4150 4150 4150
 $Comp
-L GND #PWR037
+L GND #PWR20
 U 1 1 575FF10A
 P 3650 4750
-F 0 "#PWR037" H 3650 4500 50  0001 C CNN
+F 0 "#PWR20" H 3650 4500 50  0001 C CNN
 F 1 "GND" H 3655 4577 50  0000 C CNN
 F 2 "" H 3650 4750 50  0000 C CNN
@@
 Wire Wire Line
 	4150 3750 4050 3750
-Wire Wire Line
-	4050 3750 4050 4050
-Wire Wire Line
-	4050 4050 4150 4050
-$Comp
-L +5V #PWR038
+$Comp
+L +5V #PWR19
 U 1 1 575FF10B
 P 3650 3650
-F 0 "#PWR038" H 3650 3500 50  0001 C CNN
+F 0 "#PWR19" H 3650 3500 50  0001 C CNN
 F 1 "+5V" H 3665 3823 50  0000 C CNN
 F 2 "" H 3650 3650 50  0000 C CNN
@@
 Connection ~ 3650 4250
 Wire Wire Line
-	4050 3950 4150 3950
-Connection ~ 4050 3950
-Wire Wire Line
 	3650 4550 3650 4750
 Wire Wire Line
-	3250 4650 4050 4650
-Wire Wire Line
-	6550 4225 6550 4150
-Connection ~ 6550 4150
+	4050 4650 3250 4650
 Wire Wire Line
 	3250 3850 3250 3925
@@
 	5525 4200 5525 4650
 Connection ~ 5525 4300
-Connection ~ 5250 3650
-Wire Wire Line
-	5250 3700 5250 3650
 Wire Wire Line
 	5250 3900 5250 4300
 Connection ~ 5250 4300
-Connection ~ 5525 3650
 $Comp
 L C_Small C604
@@
 Connection ~ 6000 3650
 Wire Wire Line
-	5525 3475 5525 3800
-Wire Wire Line
-	4050 4650 4050 3950
+	4050 3750 4050 4650
 Text Label 6725 4000 0    60   ~ 0
 1
@@
 -5
 Wire Wire Line
-	3250 4125 3250 4650
+	3250 4650 3250 4125
 Connection ~ 3650 4650
+Wire Wire Line
+	4150 3950 4050 3950
+Connection ~ 4050 3950
+Wire Wire Line
+	4150 4050 4050 4050
+Connection ~ 4050 4050
+Wire Wire Line
+	5150 3950 5150 4050
+Connection ~ 5150 4000
+Wire Wire Line
+	5250 3700 5250 3650
+Connection ~ 5250 3650
+Wire Wire Line
+	5525 3475 5525 3800
+Connection ~ 5525 3650
+Wire Wire Line
+	6550 4225 6550 4150
+Connection ~ 6550 4150
+Wire Wire Line
+	7800 4150 7800 4050
+Connection ~ 7800 4050
 $EndSCHEMATC
