File: GD4.sch (KiCad schematic (older format))
At the start: 19 parts, among them IC11 HCPL-316J, IC12 IXDD614PI, P6 CONN_01X03, P7 CONN_01X03

Commit message: uding HCPL-361J modified symbol
Parts:
- IC11: symbol HCPL-316J-RESCUE-gatedrive -> HCPL-316J
Connections:
- wire segments 41 -> 50
Other:
- moved on the sheet: IC12
Changed lines of the file:
@@
 EESchema Schematic File Version 2
-LIBS:gatedrive-rescue
 LIBS:power
 LIBS:device
@@
 LIBS:contrib
 LIBS:valves
-LIBS:GateDrive
+LIBS:74xgxx
+LIBS:ac-dc
+LIBS:actel
+LIBS:Altera
+LIBS:analog_devices
+LIBS:brooktre
+LIBS:cmos_ieee
+LIBS:dc-dc
+LIBS:diode
+LIBS:elec-unifil
+LIBS:ESD_Protection
+LIBS:ftdi
+LIBS:gennum
+LIBS:graphic
+LIBS:hc11
+LIBS:ir
+LIBS:Lattice
+LIBS:logo
+LIBS:maxim
+LIBS:microchip_dspic33dsc
+LIBS:microchip_pic10mcu
+LIBS:microchip_pic12mcu
+LIBS:microchip_pic16mcu
+LIBS:microchip_pic18mcu
+LIBS:microchip_pic32mcu
+LIBS:motor_drivers
+LIBS:msp430
+LIBS:nordicsemi
+LIBS:nxp_armmcu
+LIBS:onsemi
+LIBS:Oscillators
+LIBS:powerint
+LIBS:Power_Management
+LIBS:pspice
+LIBS:references
+LIBS:relays
+LIBS:rfcom
+LIBS:sensors
+LIBS:silabs
+LIBS:stm8
+LIBS:stm32
+LIBS:supertex
+LIBS:switches
+LIBS:transf
+LIBS:ttl_ieee
+LIBS:video
+LIBS:Worldsemi
+LIBS:Xicor
+LIBS:Zilog
 LIBS:gatedrive-cache
 EELAYER 25 0
@@
 L IXDD614PI-RESCUE-gatedrive IC12
 U 1 1 56EF3C27
-P 7900 5100
-F 0 "IC12" H 7900 4900 60  0000 C CNN
-F 1 "IXDD614PI" H 7950 5450 60  0000 C CNN
-F 2 "gatedrive:DIP-8_W7.62mm_LongPads" H 7900 5200 60  0001 C CNN
-F 3 "" H 7900 5200 60  0000 C CNN
-F 4 "CHINA[already bought]" H 7900 5100 60  0001 C CNN "Supplier"
-	1    7900 5100
-	1    0    0    -1
-$EndComp
-$Comp
-L HCPL-316J-RESCUE-gatedrive IC11
+P 7950 5100
+AR Path="/56EF3C27" Ref="IC12"  Part="1"
+AR Path="/56EF0560/56EF3C27" Ref="IC12"  Part="1"
+F 0 "IC12" H 7950 4900 60  0000 C CNN
+F 1 "IXDD614PI" H 8000 5450 60  0000 C CNN
+F 2 "gatedrive:DIP-8_W7.62mm_LongPads" H 7950 5200 60  0001 C CNN
+F 3 "" H 7950 5200 60  0000 C CNN
+F 4 "CHINA[already bought]" H 7950 5100 60  0001 C CNN "Supplier"
+	1    7950 5100
+	1    0    0    -1
+$EndComp
+$Comp
+L HCPL-316J IC11
 U 1 1 56EF3C28
-P 5550 4750
-F 0 "IC11" H 5550 4150 60  0000 C CNN
-F 1 "HCPL-316J" H 5300 5200 60  0000 C CNN
-F 2 "Housings_SOIC:SOIC-16_7.5x10.3mm_Pitch1.27mm" H 5550 4750 60  0001 C CNN
-F 3 "" H 5550 4750 60  0000 C CNN
-F 4 "CHINA [ already bought]" H 5550 4750 60  0001 C CNN "Supplier"
-	1    5550 4750
+P 5600 4850
+F 0 "IC11" H 5600 4250 60  0000 C CNN
+F 1 "HCPL-316J" H 5350 5350 60  0000 C CNN
+F 2 "Housings_SOIC:SOIC-16_7.5x10.3mm_Pitch1.27mm" H 5600 4850 60  0001 C CNN
+F 3 "" H 5600 4850 60  0000 C CNN
+F 4 "CHINA [ already bought]" H 5600 4850 60  0001 C CNN "Supplier"
+	1    5600 4850
 	1    0    0    -1
 $EndComp
@@
 Text GLabel 6450 4800 2    60   Input ~ 0
 15V4
-Text GLabel 7500 4850 0    60   Input ~ 0
-15V4
-Text GLabel 7500 5150 0    60   Input ~ 0
--5V4
-Text GLabel 8350 5150 2    60   Input ~ 0
+Text GLabel 7550 4850 0    60   Input ~ 0
+15V4
+Text GLabel 7550 5150 0    60   Input ~ 0
+-5V4
+Text GLabel 8300 5150 2    60   Input ~ 0
 -5V4
 Text GLabel 10200 4950 2    60   Input ~ 0
@@
 a cap to ensure soft turn-off, recommended by datasheet of hcpl.
 Wire Wire Line
-	6950 4950 7500 4950
-Wire Wire Line
-	6250 4950 6650 4950
-Wire Wire Line
-	6250 5050 6250 5150
-Wire Wire Line
-	6250 4750 6250 4850
+	6950 4950 7150 4950
+Wire Wire Line
+	7150 4950 7550 4950
+Wire Wire Line
+	5800 4950 6500 4950
+Wire Wire Line
+	6500 4950 6650 4950
+Wire Wire Line
+	5800 5050 5800 5100
+Wire Wire Line
+	5800 5100 5800 5150
+Wire Wire Line
+	5800 4750 5800 4800
+Wire Wire Line
+	5800 4800 5800 4850
 Connection ~ 6550 4100
 Wire Wire Line
-	6550 4650 6250 4650
+	6550 4650 5800 4650
 Wire Wire Line
 	6550 4100 6650 4100
 Wire Wire Line
-	6550 4050 6550 4650
+	6550 4050 6550 4100
+Wire Wire Line
+	6550 4100 6550 4650
 Connection ~ 8450 4950
 Wire Wire Line
@@
 Connection ~ 7150 4950
 Wire Wire Line
-	3625 4650 4850 4650
-Wire Wire Line
-	8350 4950 9050 4950
+	3625 4650 4000 4650
+Wire Wire Line
+	4000 4650 4900 4650
+Wire Wire Line
+	8300 4950 8450 4950
+Wire Wire Line
+	8450 4950 8900 4950
+Wire Wire Line
+	8900 4950 9050 4950
 Wire Wire Line
 	9350 4950 9450 4950
 Wire Wire Line
-	9750 4950 10200 4950
+	9750 4950 9950 4950
+Wire Wire Line
+	9950 4950 10200 4950
 Wire Wire Line
 	9750 5250 9950 5250
@@
 Connection ~ 9950 4950
 Wire Wire Line
-	8350 5050 8450 5050
+	8300 5050 8450 5050
 Wire Wire Line
 	8450 5050 8450 4950
@@
 	4400 4350 4400 4550
 Wire Wire Line
-	4400 4550 4850 4550
+	4400 4550 4900 4550
 Wire Wire Line
 	4000 4350 4000 4650
@@
 	4000 5300 4000 4750
 Wire Wire Line
-	4000 4750 4850 4750
-Wire Wire Line
-	4850 5150 4750 5150
+	4000 4750 4900 4750
+Wire Wire Line
+	4900 5150 4750 5150
 Wire Wire Line
 	4750 5150 4750 5300
 Wire Wire Line
-	4850 4850 4400 4850
+	4900 4850 4400 4850
 Wire Wire Line
 	4400 4850 4400 5300
 Wire Wire Line
-	6250 4450 6300 4450
+	5800 4450 6300 4450
 Wire Wire Line
 	6300 4450 6300 4350
@@
 	6300 5300 6300 5100
 Wire Wire Line
-	6300 5100 6250 5100
-Connection ~ 6250 5100
-Wire Wire Line
-	6250 4800 6450 4800
-Connection ~ 6250 4800
+	6300 5100 5800 5100
+Connection ~ 5800 5100
+Wire Wire Line
+	5800 4800 6450 4800
+Connection ~ 5800 4800
 Wire Wire Line
 	8900 5250 9450 5250
@@
 Wire Wire Line
 	6500 5000 6500 4950
-Text GLabel 8350 4850 2    60   Input ~ 0
+Text GLabel 8300 4850 2    60   Input ~ 0
 15V4
 Text GLabel 7175 5075 3    60   Input ~ 0
 15V4
 Wire Wire Line
-	7500 5050 7175 5050
+	7550 5050 7175 5050
 Wire Wire Line
 	7175 5050 7175 5075
 Text HLabel 900  3800 3    60   Input ~ 0
 T4
-Text HLabel 4850 4450 0    60   Input ~ 0
+Text HLabel 4900 4450 0    60   Input ~ 0
 T4
 Text GLabel 900  2650 3    60   Input ~ 0
@@
 Text GLabel 4400 5300 3    60   Input ~ 0
 ~RST
-Text GLabel 4850 4950 0    60   Input ~ 0
+Text GLabel 4900 4950 0    60   Input ~ 0
 ~FAULT
 Text GLabel 3625 4350 1    60   Input ~ 0

Commit message: cleaning the schematic
Connections:
- wire segments 50 -> 41
Changed lines of the file:
@@
 a cap to ensure soft turn-off, recommended by datasheet of hcpl.
 Wire Wire Line
-	6950 4950 7150 4950
+	6950 4950 7550 4950
 Wire Wire Line
-	7150 4950 7550 4950
+	5800 4950 6650 4950
 Wire Wire Line
-	5800 4950 6500 4950
+	5800 5050 5800 5150
 Wire Wire Line
-	6500 4950 6650 4950
-Wire Wire Line
-	5800 5050 5800 5100
-Wire Wire Line
-	5800 5100 5800 5150
-Wire Wire Line
-	5800 4750 5800 4800
-Wire Wire Line
-	5800 4800 5800 4850
+	5800 4750 5800 4850
 Connection ~ 6550 4100
 Wire Wire Line
@@
 	6550 4100 6650 4100
 Wire Wire Line
-	6550 4050 6550 4100
-Wire Wire Line
-	6550 4100 6550 4650
+	6550 4050 6550 4650
 Connection ~ 8450 4950
 Wire Wire Line
@@
 Connection ~ 7150 4950
 Wire Wire Line
-	3625 4650 4000 4650
+	3625 4650 4900 4650
 Wire Wire Line
-	4000 4650 4900 4650
-Wire Wire Line
-	8300 4950 8450 4950
-Wire Wire Line
-	8450 4950 8900 4950
-Wire Wire Line
-	8900 4950 9050 4950
+	8300 4950 9050 4950
 Wire Wire Line
 	9350 4950 9450 4950
 Wire Wire Line
-	9750 4950 9950 4950
-Wire Wire Line
-	9950 4950 10200 4950
+	9750 4950 10200 4950
 Wire Wire Line
 	9750 5250 9950 5250

Commit message: completion of the layout, initial layout of the protection circuit, reducing number of circuit to 7
Parts:
- C36, C37, C38, C40, C41, C42: footprint Capacitors_ThroughHole:C_Disc_D3_P2.5 -> gatedrive:C_Disc
- D11: footprint Diodes_ThroughHole:Diode_DO-201AD_Horizontal_RM15 -> Diodes_ThroughHole:Diode_DO-41_SOD81_Horizontal_RM10
- R31: footprint Resistors_ThroughHole:Resistor_Vertical_RM5mm -> Resistors_ThroughHole:Resistor_Horizontal_RM10mm
- R35, R36: footprint Resistors_ThroughHole:Resistor_Horizontal_RM20mm -> gatedrive:Resistor_multi
Changed lines of the file:
@@
 EESchema Schematic File Version 2
+LIBS:Symbols_DCDC-ACDC-Converter_RevC_20Jul2012
+LIBS:Symbols_EN60617_13Mar2013
+LIBS:Symbols_EN60617-10_HF-Radio_DRAFT_12Sep2013
+LIBS:Symbols_ICs-Diskrete_RevD10
+LIBS:Symbols_ICs-Opto_RevB_16Sep2013
+LIBS:Symbols_Microcontroller_Philips-NXP_RevA_06Oct2013
+LIBS:SymbolsSimilarEN60617+oldDIN617-RevE8
+LIBS:Symbols_Socket-DIN41612_RevA
+LIBS:Symbols_Transformer-Diskrete_RevA
 LIBS:power
 LIBS:device
@@
 $Descr A4 11693 8268
 encoding utf-8
-Sheet 7 10
+Sheet 7 9
 Title "IGBT GATE DRIVE SCHEMATIC."
 Date "2016-03-02"
@@
 F 0 "D11" H 7150 3976 50  0000 C CNN
 F 1 "RGPO2-20" H 7150 3900 50  0000 C CNN
-F 2 "Diodes_ThroughHole:Diode_DO-201AD_Horizontal_RM15" H 7150 4100 50  0001 C CNN
+F 2 "Diodes_ThroughHole:Diode_DO-41_SOD81_Horizontal_RM10" H 7150 4100 50  0001 C CNN
 F 3 "" H 7150 4100 50  0000 C CNN
 F 4 "El-Amir" H 7150 4100 60  0001 C CNN "Supplier"
@@
 F 0 "R31" V 3525 4500 50  0000 C CNN
 F 1 "10K" V 3625 4500 50  0000 C CNN
-F 2 "Resistors_ThroughHole:Resistor_Vertical_RM5mm" V 3555 4500 50  0001 C CNN
+F 2 "Resistors_ThroughHole:Resistor_Horizontal_RM10mm" V 3555 4500 50  0001 C CNN
 F 3 "" H 3625 4500 50  0000 C CNN
 F 4 "EL AMIR" H 3625 4500 60  0001 C CNN "Supplier"
@@
 F 0 "C36" H 4150 2150 50  0000 C CNN
 F 1 "0.1uF" H 4250 2050 50  0000 C CNN
-F 2 "Capacitors_ThroughHole:C_Disc_D3_P2.5" H 4488 2000 50  0001 C CNN
+F 2 "gatedrive:C_Disc" H 4488 2000 50  0001 C CNN
 F 3 "" H 4450 2150 50  0000 C CNN
 F 4 "EL AMIR" H 4450 2150 60  0001 C CNN "Supplier"
@@
 F 0 "C38" H 7000 3900 50  0000 C CNN
 F 1 "100pF" H 6800 3900 50  0000 C CNN
-F 2 "Capacitors_ThroughHole:C_Disc_D3_P2.5" H 6588 3750 50  0001 C CNN
+F 2 "gatedrive:C_Disc" H 6588 3750 50  0001 C CNN
 F 3 "" H 6550 3900 50  0000 C CNN
 	1    6550 3900
@@
 F 0 "C42" H 8450 2150 50  0000 C CNN
 F 1 "0.1uF" H 8450 2050 50  0000 C CNN
-F 2 "Capacitors_ThroughHole:C_Disc_D3_P2.5" H 8888 2000 50  0001 C CNN
+F 2 "gatedrive:C_Disc" H 8888 2000 50  0001 C CNN
 F 3 "" H 8850 2150 50  0000 C CNN
 	1    8850 2150
@@
 F 0 "C41" H 7400 2150 50  0000 C CNN
 F 1 "0.1uF" H 7400 2050 50  0000 C CNN
-F 2 "Capacitors_ThroughHole:C_Disc_D3_P2.5" H 7788 2000 50  0001 C CNN
+F 2 "gatedrive:C_Disc" H 7788 2000 50  0001 C CNN
 F 3 "" H 7750 2150 50  0000 C CNN
 	1    7750 2150
@@
 F 0 "C37" H 5150 2150 50  0000 C CNN
 F 1 "0.1uF" H 5150 2050 50  0000 C CNN
-F 2 "Capacitors_ThroughHole:C_Disc_D3_P2.5" H 5538 2000 50  0001 C CNN
+F 2 "gatedrive:C_Disc" H 5538 2000 50  0001 C CNN
 F 3 "" H 5500 2150 50  0000 C CNN
 	1    5500 2150
@@
 LEFT OPEN OR CONNECTED TO THE VCC.
 $Comp
-L PWR_FLAG #FLG036
+L PWR_FLAG #FLG022
 U 1 1 56EF3C35
 P 1300 3800
-F 0 "#FLG036" H 1300 3895 50  0001 C CNN
+F 0 "#FLG022" H 1300 3895 50  0001 C CNN
 F 1 "PWR_FLAG" H 1300 4024 50  0000 C CNN
 F 2 "" H 1300 3800 50  0000 C CNN
@@
 $EndComp
 $Comp
-L PWR_FLAG #FLG037
+L PWR_FLAG #FLG023
 U 1 1 56EF3C36
 P 1750 3800
-F 0 "#FLG037" H 1750 3895 50  0001 C CNN
+F 0 "#FLG023" H 1750 3895 50  0001 C CNN
 F 1 "PWR_FLAG" H 1750 4024 50  0000 C CNN
 F 2 "" H 1750 3800 50  0000 C CNN
@@
 $EndComp
 $Comp
-L PWR_FLAG #FLG038
+L PWR_FLAG #FLG024
 U 1 1 56EF3C37
 P 1750 2650
-F 0 "#FLG038" H 1750 2745 50  0001 C CNN
+F 0 "#FLG024" H 1750 2745 50  0001 C CNN
 F 1 "PWR_FLAG" H 1750 2874 50  0000 C CNN
 F 2 "" H 1750 2650 50  0000 C CNN
@@
 $EndComp
 $Comp
-L PWR_FLAG #FLG039
+L PWR_FLAG #FLG025
 U 1 1 56EF3C38
 P 900 2650
-F 0 "#FLG039" H 900 2745 50  0001 C CNN
+F 0 "#FLG025" H 900 2745 50  0001 C CNN
 F 1 "PWR_FLAG" H 900 2874 50  0000 C CNN
 F 2 "" H 900 2650 50  0000 C CNN
@@
 $EndComp
 $Comp
-L PWR_FLAG #FLG040
+L PWR_FLAG #FLG026
 U 1 1 56EF3C39
 P 1300 2650
-F 0 "#FLG040" H 1300 2745 50  0001 C CNN
+F 0 "#FLG026" H 1300 2745 50  0001 C CNN
 F 1 "PWR_FLAG" H 1300 2874 50  0000 C CNN
 F 2 "" H 1300 2650 50  0000 C CNN
@@
 $EndComp
 $Comp
-L PWR_FLAG #FLG041
+L PWR_FLAG #FLG027
 U 1 1 56EF3C3A
 P 900 3800
-F 0 "#FLG041" H 900 3895 50  0001 C CNN
+F 0 "#FLG027" H 900 3895 50  0001 C CNN
 F 1 "PWR_FLAG" H 900 4024 50  0000 C CNN
 F 2 "" H 900 3800 50  0000 C CNN
@@
 F 0 "C40" H 7390 4630 50  0000 C CNN
 F 1 "10nF" H 7400 4550 50  0000 C CNN
-F 2 "Capacitors_ThroughHole:C_Disc_D3_P2.5" H 7188 4450 50  0001 C CNN
+F 2 "gatedrive:C_Disc" H 7188 4450 50  0001 C CNN
 F 3 "" H 7150 4600 50  0000 C CNN
 	1    7150 4600
@@
 F 0 "R35" V 9600 4980 50  0000 C CNN
 F 1 "60" V 9500 4950 50  0000 C CNN
-F 2 "Resistors_ThroughHole:Resistor_Horizontal_RM20mm" V 9530 4950 50  0001 C CNN
+F 2 "gatedrive:Resistor_multi" V 9530 4950 50  0001 C CNN
 F 3 "" H 9600 4950 50  0000 C CNN
 F 4 "Al amir" H 9600 4950 60  0001 C CNN "Supplier"
@@
 F 0 "R36" V 9600 5240 50  0000 C CNN
 F 1 "30ohm ,0.5W" V 9500 5250 50  0000 C CNN
-F 2 "Resistors_ThroughHole:Resistor_Horizontal_RM20mm" V 9530 5250 50  0001 C CNN
+F 2 "gatedrive:Resistor_multi" V 9530 5250 50  0001 C CNN
 F 3 "" H 9600 5250 50  0000 C CNN
 F 4 "Supplier_name" H 9600 5250 60  0001 C CNN "Supplier"
@@
 	6950 4100 7000 4100
 $Comp
-L PWR_FLAG #FLG042
+L PWR_FLAG #FLG028
 U 1 1 56EF3C41
 P 1475 3050
-F 0 "#FLG042" H 1475 3145 50  0001 C CNN
+F 0 "#FLG028" H 1475 3145 50  0001 C CNN
 F 1 "PWR_FLAG" V 1625 3050 50  0000 C CNN
 F 2 "" H 1475 3050 50  0000 C CNN

Commit message: yet another enhancements .
the protection section still is incomplete.
Parts:
- IC12: symbol IXDD614PI-RESCUE-gatedrive -> IXDD614PI
Connections:
- wire segments 41 -> 50
Other:
- moved on the sheet: IC11
Changed lines of the file:
@@
 $Descr A4 11693 8268
 encoding utf-8
-Sheet 7 9
+Sheet 5 9
 Title "IGBT GATE DRIVE SCHEMATIC."
 Date "2016-03-02"
@@
 $EndDescr
 $Comp
-L IXDD614PI-RESCUE-gatedrive IC12
+L IXDD614PI IC12
 U 1 1 56EF3C27
-P 7950 5100
+P 7950 4950
 AR Path="/56EF3C27" Ref="IC12"  Part="1"
 AR Path="/56EF0560/56EF3C27" Ref="IC12"  Part="1"
-F 0 "IC12" H 7950 4900 60  0000 C CNN
-F 1 "IXDD614PI" H 8000 5450 60  0000 C CNN
-F 2 "gatedrive:DIP-8_W7.62mm_LongPads" H 7950 5200 60  0001 C CNN
-F 3 "" H 7950 5200 60  0000 C CNN
-F 4 "CHINA[already bought]" H 7950 5100 60  0001 C CNN "Supplier"
-	1    7950 5100
+F 0 "IC12" H 7950 4750 60  0000 C CNN
+F 1 "IXDD614PI" H 8000 5300 60  0000 C CNN
+F 2 "gatedrive:DIP-8_W7.62mm_LongPads" H 7950 5050 60  0001 C CNN
+F 3 "" H 7950 5050 60  0000 C CNN
+F 4 "CHINA[already bought]" H 7950 4950 60  0001 C CNN "Supplier"
+	1    7950 4950
 	1    0    0    -1
 $EndComp
@@
 L HCPL-316J IC11
 U 1 1 56EF3C28
-P 5600 4850
-F 0 "IC11" H 5600 4250 60  0000 C CNN
-F 1 "HCPL-316J" H 5350 5350 60  0000 C CNN
-F 2 "Housings_SOIC:SOIC-16_7.5x10.3mm_Pitch1.27mm" H 5600 4850 60  0001 C CNN
-F 3 "" H 5600 4850 60  0000 C CNN
-F 4 "CHINA [ already bought]" H 5600 4850 60  0001 C CNN "Supplier"
-	1    5600 4850
+P 5300 4750
+AR Path="/56EF3C28" Ref="IC11"  Part="1"
+AR Path="/56EF0560/56EF3C28" Ref="IC11"  Part="1"
+F 0 "IC11" H 5300 4150 60  0000 C CNN
+F 1 "HCPL-316J" H 5050 5250 60  0000 C CNN
+F 2 "Housings_SOIC:SOIC-16_7.5x10.3mm_Pitch1.27mm" H 5300 4750 60  0001 C CNN
+F 3 "" H 5300 4750 60  0000 C CNN
+F 4 "CHINA [ already bought]" H 5300 4750 60  0001 C CNN "Supplier"
+	1    5300 4750
 	1    0    0    -1
 $EndComp
@@
 Text GLabel 7550 5150 0    60   Input ~ 0
 -5V4
-Text GLabel 8300 5150 2    60   Input ~ 0
+Text GLabel 8350 5150 2    60   Input ~ 0
 -5V4
 Text GLabel 10200 4950 2    60   Input ~ 0
@@
 a cap to ensure soft turn-off, recommended by datasheet of hcpl.
 Wire Wire Line
-	6950 4950 7550 4950
-Wire Wire Line
-	5800 4950 6650 4950
-Wire Wire Line
-	5800 5050 5800 5150
-Wire Wire Line
-	5800 4750 5800 4850
+	6950 4950 7150 4950
+Wire Wire Line
+	7150 4950 7550 4950
+Wire Wire Line
+	5800 4950 6500 4950
+Wire Wire Line
+	6500 4950 6650 4950
+Wire Wire Line
+	5800 5050 5800 5100
+Wire Wire Line
+	5800 5100 5800 5150
+Wire Wire Line
+	5800 4750 5800 4800
+Wire Wire Line
+	5800 4800 5800 4850
 Connection ~ 6550 4100
 Wire Wire Line
@@
 	6550 4100 6650 4100
 Wire Wire Line
-	6550 4050 6550 4650
+	6550 4050 6550 4100
+Wire Wire Line
+	6550 4100 6550 4650
 Connection ~ 8450 4950
 Wire Wire Line
@@
 Connection ~ 7150 4950
 Wire Wire Line
-	3625 4650 4900 4650
-Wire Wire Line
-	8300 4950 9050 4950
+	3625 4650 4000 4650
+Wire Wire Line
+	4000 4650 4800 4650
+Wire Wire Line
+	8350 4950 8450 4950
+Wire Wire Line
+	8450 4950 8900 4950
+Wire Wire Line
+	8900 4950 9050 4950
 Wire Wire Line
 	9350 4950 9450 4950
 Wire Wire Line
-	9750 4950 10200 4950
+	9750 4950 9950 4950
+Wire Wire Line
+	9950 4950 10200 4950
 Wire Wire Line
 	9750 5250 9950 5250
@@
 Connection ~ 9950 4950
 Wire Wire Line
-	8300 5050 8450 5050
+	8350 5050 8450 5050
 Wire Wire Line
 	8450 5050 8450 4950
@@
 	4400 4350 4400 4550
 Wire Wire Line
-	4400 4550 4900 4550
+	4400 4550 4800 4550
 Wire Wire Line
 	4000 4350 4000 4650
@@
 	4000 5300 4000 4750
 Wire Wire Line
-	4000 4750 4900 4750
-Wire Wire Line
-	4900 5150 4750 5150
+	4000 4750 4800 4750
+Wire Wire Line
+	4800 5150 4750 5150
 Wire Wire Line
 	4750 5150 4750 5300
 Wire Wire Line
-	4900 4850 4400 4850
+	4800 4850 4400 4850
 Wire Wire Line
 	4400 4850 4400 5300
@@
 Wire Wire Line
 	6500 5000 6500 4950
-Text GLabel 8300 4850 2    60   Input ~ 0
+Text GLabel 8350 4850 2    60   Input ~ 0
 15V4
 Text GLabel 7175 5075 3    60   Input ~ 0
@@
 Text HLabel 900  3800 3    60   Input ~ 0
 T4
-Text HLabel 4900 4450 0    60   Input ~ 0
+Text HLabel 4800 4450 0    60   Input ~ 0
 T4
 Text GLabel 900  2650 3    60   Input ~ 0
@@
 Text GLabel 4400 5300 3    60   Input ~ 0
 ~RST
-Text GLabel 4900 4950 0    60   Input ~ 0
+Text GLabel 4800 4950 0    60   Input ~ 0
 ~FAULT
 Text GLabel 3625 4350 1    60   Input ~ 0

Commit message: packup
Parts:
- removed C36, C37, C41, C42: 0.1uF, gatedrive:C_Disc, symbol CP1
- removed C38: 100pF, gatedrive:C_Disc, symbol CP1
- removed C39: 330pF, Capacitors_ThroughHole:C_Disc_D3_P2.5, symbol CP1
- removed C40: 10nF, gatedrive:C_Disc, symbol CP1
- removed D11: RGPO2-20, Diodes_ThroughHole:Diode_DO-41_SOD81_Horizontal_RM10, symbol D
- removed D12: ~, Diodes_ThroughHole:Diode_DO-201AD_Horizontal_RM15, symbol D
- removed IC11: HCPL-316J, Housings_SOIC:SOIC-16_7.5x10.3mm_Pitch1.27mm, symbol HCPL-316J
- removed IC12: IXDD614PI, gatedrive:DIP-8_W7.62mm_LongPads, symbol IXDD614PI
- removed P6, P7: CONN_01X03, Pin_Headers:Pin_Header_Angled_1x03, symbol CONN_01X03
- removed R31: 10K, Resistors_ThroughHole:Resistor_Horizontal_RM10mm, symbol R
- removed R32: 25K, Resistors_ThroughHole:Resistor_Horizontal_RM10mm, symbol R
- removed R33, R34: 100, Resistors_ThroughHole:Resistor_Horizontal_RM10mm, symbol R
- removed R35: 60, gatedrive:Resistor_multi, symbol R
- removed R36: 30ohm ,0.5W, gatedrive:Resistor_multi, symbol R
- added C501, C503, C504, C505: 0.1uF, gatedrive:C_Disc, symbol C_Small
- added C502: 330pF, gatedrive:C_Disc, symbol C_Small
- added C506: 100pF, gatedrive:C_Disc, symbol C_Small
- added C507: 10nF, gatedrive:C_Disc, symbol C_Small
- added D501: RGPO2-20, Diodes_ThroughHole:Diode_DO-41_SOD81_Horizontal_RM10, symbol D
- added D502: ~, Diodes_ThroughHole:Diode_DO-201AD_Horizontal_RM15, symbol D
- added IC501: HCPL-316J, Housings_SOIC:SOIC-16_7.5x10.3mm_Pitch1.27mm, symbol HCPL-316J
- added IC502: IXDD614PI, gatedrive:DIP-8_W7.62mm_LongPads, symbol IXDD614PI
- added P501, P502: CONN_01X03, gatedrive:conn, symbol CONN_01X03
- added R501: 10K, Resistors_ThroughHole:Resistor_Horizontal_RM10mm, symbol R_Small
- added R502: 25K, Resistors_ThroughHole:Resistor_Horizontal_RM10mm, symbol R_Small
- added R503, R504: 100, Resistors_ThroughHole:Resistor_Horizontal_RM10mm, symbol R_Small
- added R505: 60, gatedrive:Resistor_multi, symbol R_Small
- added R506: 30ohm ,0.5W, gatedrive:Resistor_multi, symbol R_Small
Connections:
- net 15V4: now also C504.2, C505.1, IC501.12 (Vc), IC501.13 (Vcc2), IC502.1 (VCC), IC502.3 (EN), IC502.8 (VCC), P501.2 (P2)
- net COM4: now also C503.2, C504.1, C506.2, IC501.16 (VE), P501.1 (P1), P502.3 (P3)
- net G4: now also P502.1 (P1), R505.2, R506.2
- net T4: now also IC501.1 (Vin+)
- net ~FAULT: now also C502.1, IC501.6 (~FAULT), R501.1
- net ~RST: now also IC501.5 (~RESET)
- new net: IC501.11 (Vout), R502.2, R504.2
- new net: C506.1, IC501.14 (DESAT), R503.1
- new net: C507.1, IC502.2 (IN), R504.1
- new net: D501.2 (A), R503.2
- new net: D502.1 (K), R505.1
- new net: D502.2 (A), IC502.6 (OUT), IC502.7 (OUT), R506.1
- new net +5V: C501.1, IC501.3 (Vcc1), R501.2
- new net -5v4: C503.1, C505.2, C507.2, IC501.10 (VEE), IC501.9 (VEE), IC502.4 (GND), IC502.5 (GND), P501.3 (P3), R502.1
- new net GND: C501.2, C502.2, IC501.2 (Vin-), IC501.4 (GND1), IC501.8 (Vled1-)
- new net c4: D501.1 (K), P502.2 (P2)
Other:
- note added: "5 volt is the vcc of the microcontroller.\n"
- note added: "GND is the ground of the microcontroller.\n"
- note added: "IN PIN IS LEFT OPEN OR CONNECTED TO THE VCC."
- note added: "a cap to ensure soft turn-off,\n recommended by datasheet of hcpl."
- note removed: "Fault pull-up resistor."
- note removed: "GND1 is the ground of the microcontroller.\n"
- note removed: "I'M USING GLOBAL LABELS INSTEAD OF LOCAL LABELS AS THEY LOOK NEATER, LOL."
- note removed: "LEFT OPEN OR CONNECTED TO THE VCC."
- note removed: "MICSUPP is 5 volt from the vcc of the microcontroller.\n"
- note removed: "a cap to ensure soft turn-off, recommended by datasheet of hcpl."
