File: GD5.sch (KiCad schematic (older format))
At the start: 19 parts, among them IC7 HCPL-316J, IC8 IXDD614PI, P4 CONN_01X03, P5 CONN_01X03

Commit message: packup
Parts:
- removed C22, C23, C27, C28: 0.1uF, gatedrive:C_Disc, symbol CP1
- removed C24: 100pF, gatedrive:C_Disc, symbol CP1
- removed C25: 330pF, Capacitors_ThroughHole:C_Disc_D3_P2.5, symbol CP1
- removed C26: 10nF, gatedrive:C_Disc, symbol CP1
- removed D7: RGPO2-20, Diodes_ThroughHole:Diode_DO-41_SOD81_Horizontal_RM10, symbol D
- removed D8: ~, Diodes_ThroughHole:Diode_DO-201AD_Horizontal_RM15, symbol D
- removed IC7: HCPL-316J, Housings_SOIC:SOIC-16_7.5x10.3mm_Pitch1.27mm, symbol HCPL-316J
- removed IC8: IXDD614PI, gatedrive:DIP-8_W7.62mm_LongPads, symbol IXDD614PI
- removed P4, P5: CONN_01X03, Pin_Headers:Pin_Header_Angled_1x03, symbol CONN_01X03
- removed R19: 10K, Resistors_ThroughHole:Resistor_Horizontal_RM10mm, symbol R
- removed R20: 25K, Resistors_ThroughHole:Resistor_Horizontal_RM10mm, symbol R
- removed R21, R22: 100, Resistors_ThroughHole:Resistor_Horizontal_RM10mm, symbol R
- removed R23: 60, gatedrive:Resistor_multi, symbol R
- removed R24: 30ohm ,0.5W, gatedrive:Resistor_multi, symbol R
- added C401, C403, C404, C405: 0.1uF, gatedrive:C_Disc, symbol C_Small
- added C402: 330pF, gatedrive:C_Disc, symbol C_Small
- added C406: 100pF, gatedrive:C_Disc, symbol C_Small
- added C407: 10nF, gatedrive:C_Disc, symbol C_Small
- added D401: RGPO2-20, Diodes_ThroughHole:Diode_DO-41_SOD81_Horizontal_RM10, symbol D
- added D402: ~, Diodes_ThroughHole:Diode_DO-201AD_Horizontal_RM15, symbol D
- added IC401: HCPL-316J, Housings_SOIC:SOIC-16_7.5x10.3mm_Pitch1.27mm, symbol HCPL-316J
- added IC402: IXDD614PI, gatedrive:DIP-8_W7.62mm_LongPads, symbol IXDD614PI
- added P401, P402: CONN_01X03, gatedrive:conn, symbol CONN_01X03
- added R401: 10K, Resistors_ThroughHole:Resistor_Horizontal_RM10mm, symbol R_Small
- added R402: 25K, Resistors_ThroughHole:Resistor_Horizontal_RM10mm, symbol R_Small
- added R403, R404: 100, Resistors_ThroughHole:Resistor_Horizontal_RM10mm, symbol R_Small
- added R405: 60, gatedrive:Resistor_multi, symbol R_Small
- added R406: 30ohm ,0.5W, gatedrive:Resistor_multi, symbol R_Small
Connections:
- net 15V5: now also C404.2, C405.1, IC401.12 (Vc), IC401.13 (Vcc2), IC402.1 (VCC), IC402.3 (EN), IC402.8 (VCC), P401.2 (P2)
- net COM5: now also C403.2, C404.1, C406.2, IC401.16 (VE), P401.1 (P1), P402.3 (P3)
- net G5: now also P402.1 (P1), R405.2, R406.2
- net T5: now also IC401.1 (Vin+)
- net ~FAULT: now also C402.1, IC401.6 (~FAULT), R401.1
- net ~RST: now also IC401.5 (~RESET)
- new net: IC401.11 (Vout), R402.2, R404.2
- new net: C406.1, IC401.14 (DESAT), R403.1
- new net: C407.1, IC402.2 (IN), R404.1
- new net: D401.2 (A), R403.2
- new net: D402.1 (K), R405.1
- new net: D402.2 (A), IC402.6 (OUT), IC402.7 (OUT), R406.1
- new net +5V: C401.1, IC401.3 (Vcc1), R401.2
- new net -5v5: C403.1, C405.2, C407.2, IC401.10 (VEE), IC401.9 (VEE), IC402.4 (GND), IC402.5 (GND), P401.3 (P3), R402.1
- new net GND: C401.2, C402.2, IC401.2 (Vin-), IC401.4 (GND1), IC401.8 (Vled1-)
- new net c5: D401.1 (K), P402.2 (P2)
Other:
- note added: "5 volt is the vcc of the microcontroller.\n"
- note added: "GND is the ground of the microcontroller.\n"
- note added: "IN PIN IS LEFT OPEN OR CONNECTED TO THE VCC."
- note added: "a cap to ensure soft turn-off,\n recommended by datasheet of hcpl."
- note removed: "Fault pull-up resistor."
- note removed: "GND1 is the ground of the microcontroller.\n"
- note removed: "I'M USING GLOBAL LABELS INSTEAD OF LOCAL LABELS AS THEY LOOK NEATER, LOL."
- note removed: "LEFT OPEN OR CONNECTED TO THE VCC."
- note removed: "MICSUPP is 5 volt from the vcc of the microcontroller.\n"
- note removed: "a cap to ensure soft turn-off, recommended by datasheet of hcpl."

Commit message: parting the protection from the GD
Connections:
- net 15V5: now also P401.1 (P1); no longer P401.2 (P2)
- net COM5: now also P401.2 (P2); no longer P401.1 (P1)
Changed lines of the file:
@@
 IN PIN IS LEFT OPEN OR CONNECTED TO THE VCC.
 $Comp
-L PWR_FLAG #FLG021
+L PWR_FLAG #FLG13
 U 1 1 575FFB5F
 P 1300 3800
-F 0 "#FLG021" H 1300 3895 50  0001 C CNN
+F 0 "#FLG13" H 1300 3895 50  0001 C CNN
 F 1 "PWR_FLAG" H 1300 4024 50  0000 C CNN
 F 2 "" H 1300 3800 50  0000 C CNN
@@
 $EndComp
 $Comp
-L PWR_FLAG #FLG022
+L PWR_FLAG #FLG14
 U 1 1 575FFB60
 P 1750 3800
-F 0 "#FLG022" H 1750 3895 50  0001 C CNN
+F 0 "#FLG14" H 1750 3895 50  0001 C CNN
 F 1 "PWR_FLAG" H 1750 4024 50  0000 C CNN
 F 2 "" H 1750 3800 50  0000 C CNN
@@
 $EndComp
 $Comp
-L PWR_FLAG #FLG023
+L PWR_FLAG #FLG12
 U 1 1 575FFB63
 P 1300 2650
-F 0 "#FLG023" H 1300 2745 50  0001 C CNN
+F 0 "#FLG12" H 1300 2745 50  0001 C CNN
 F 1 "PWR_FLAG" H 1300 2874 50  0000 C CNN
 F 2 "" H 1300 2650 50  0000 C CNN
@@
 $EndComp
 $Comp
-L PWR_FLAG #FLG024
+L PWR_FLAG #FLG11
 U 1 1 575FFB64
 P 900 3800
-F 0 "#FLG024" H 900 3895 50  0001 C CNN
+F 0 "#FLG11" H 900 3895 50  0001 C CNN
 F 1 "PWR_FLAG" H 900 4024 50  0000 C CNN
 F 2 "" H 900 3800 50  0000 C CNN
@@
 	-1   0    0    1
 $EndComp
+Text GLabel 1550 4775 2    60   Input ~ 0
+COM5
 Text GLabel 1550 4875 2    60   Input ~ 0
-COM5
-Text GLabel 1550 4775 2    60   Input ~ 0
 15V5
 Text GLabel 1550 5425 2    60   Input ~ 0
@@
 	3975 4150 4150 4150
 $Comp
-L GND #PWR025
+L GND #PWR16
 U 1 1 575FFB6D
 P 3650 4750
-F 0 "#PWR025" H 3650 4500 50  0001 C CNN
+F 0 "#PWR16" H 3650 4500 50  0001 C CNN
 F 1 "GND" H 3655 4577 50  0000 C CNN
 F 2 "" H 3650 4750 50  0000 C CNN
@@
 	4050 4050 4150 4050
 $Comp
-L +5V #PWR026
+L +5V #PWR15
 U 1 1 575FFB6E
 P 3650 3650
-F 0 "#PWR026" H 3650 3500 50  0001 C CNN
+F 0 "#PWR15" H 3650 3500 50  0001 C CNN
 F 1 "+5V" H 3665 3823 50  0000 C CNN
 F 2 "" H 3650 3650 50  0000 C CNN
