File: GD6.sch (KiCad schematic (older format))
At the start: 19 parts, among them IC301 HCPL-316J, IC302 IXDD614PI, P301 CONN_01X03, P302 CONN_01X03

Commit message: parting the protection from the GD
Connections:
- net 15V6: now also P301.1 (P1); no longer P301.2 (P2)
- net COM6: now also P301.2 (P2); no longer P301.1 (P1)
Changed lines of the file:
@@
 IN PIN IS LEFT OPEN OR CONNECTED TO THE VCC.
 $Comp
-L PWR_FLAG #FLG015
+L PWR_FLAG #FLG9
 U 1 1 575FFF8C
 P 1300 3800
-F 0 "#FLG015" H 1300 3895 50  0001 C CNN
+F 0 "#FLG9" H 1300 3895 50  0001 C CNN
 F 1 "PWR_FLAG" H 1300 4024 50  0000 C CNN
 F 2 "" H 1300 3800 50  0000 C CNN
@@
 $EndComp
 $Comp
-L PWR_FLAG #FLG016
+L PWR_FLAG #FLG10
 U 1 1 575FFF8D
 P 1750 3800
-F 0 "#FLG016" H 1750 3895 50  0001 C CNN
+F 0 "#FLG10" H 1750 3895 50  0001 C CNN
 F 1 "PWR_FLAG" H 1750 4024 50  0000 C CNN
 F 2 "" H 1750 3800 50  0000 C CNN
@@
 $EndComp
 $Comp
-L PWR_FLAG #FLG017
+L PWR_FLAG #FLG8
 U 1 1 575FFF90
 P 1300 2650
-F 0 "#FLG017" H 1300 2745 50  0001 C CNN
+F 0 "#FLG8" H 1300 2745 50  0001 C CNN
 F 1 "PWR_FLAG" H 1300 2874 50  0000 C CNN
 F 2 "" H 1300 2650 50  0000 C CNN
@@
 $EndComp
 $Comp
-L PWR_FLAG #FLG018
+L PWR_FLAG #FLG7
 U 1 1 575FFF91
 P 900 3800
-F 0 "#FLG018" H 900 3895 50  0001 C CNN
+F 0 "#FLG7" H 900 3895 50  0001 C CNN
 F 1 "PWR_FLAG" H 900 4024 50  0000 C CNN
 F 2 "" H 900 3800 50  0000 C CNN
@@
 	-1   0    0    1
 $EndComp
+Text GLabel 1550 4775 2    60   Input ~ 0
+COM6
 Text GLabel 1550 4875 2    60   Input ~ 0
-COM6
-Text GLabel 1550 4775 2    60   Input ~ 0
 15V6
 Text GLabel 1550 5425 2    60   Input ~ 0
@@
 	3975 4150 4150 4150
 $Comp
-L GND #PWR019
+L GND #PWR14
 U 1 1 575FFF9A
 P 3650 4750
-F 0 "#PWR019" H 3650 4500 50  0001 C CNN
+F 0 "#PWR14" H 3650 4500 50  0001 C CNN
 F 1 "GND" H 3655 4577 50  0000 C CNN
 F 2 "" H 3650 4750 50  0000 C CNN
@@
 	4050 4050 4150 4050
 $Comp
-L +5V #PWR020
+L +5V #PWR13
 U 1 1 575FFF9B
 P 3650 3650
-F 0 "#PWR020" H 3650 3500 50  0001 C CNN
+F 0 "#PWR13" H 3650 3500 50  0001 C CNN
 F 1 "+5V" H 3665 3823 50  0000 C CNN
 F 2 "" H 3650 3650 50  0000 C CNN
