File: GD7.sch (KiCad schematic (older format))
At the start: 19 parts, among them IC3 HCPL-316J, IC4 IXDD614PI, P10 CONN_01X03, P11 CONN_01X03

Commit message: packup
Parts:
- removed C10: 100pF, gatedrive:C_Disc, symbol CP1
- removed C11: 330pF, gatedrive:C_Disc, symbol CP1
- removed C12: 10nF, gatedrive:C_Disc, symbol CP1
- removed C13, C14, C8, C9: 0.1uF, gatedrive:C_Disc, symbol CP1
- removed D3: RGPO2-20, Diodes_ThroughHole:Diode_DO-41_SOD81_Horizontal_RM10, symbol D
- removed D4: ~, Diodes_ThroughHole:Diode_DO-201AD_Horizontal_RM15, symbol D
- removed IC3: HCPL-316J, Housings_SOIC:SOIC-16_7.5x10.3mm_Pitch1.27mm, symbol HCPL-316J
- removed IC4: IXDD614PI, gatedrive:DIP-8_W7.62mm_LongPads, symbol IXDD614PI
- removed P10, P11: CONN_01X03, Pin_Headers:Pin_Header_Angled_1x03, symbol CONN_01X03
- removed R10, R9: 100, Resistors_ThroughHole:Resistor_Horizontal_RM10mm, symbol R
- removed R11: 60, gatedrive:Resistor_multi, symbol R
- removed R12: 30ohm ,0.5W, gatedrive:Resistor_multi, symbol R
- removed R7: 10K, Resistors_ThroughHole:Resistor_Horizontal_RM10mm, symbol R
- removed R8: 25K, Resistors_ThroughHole:Resistor_Horizontal_RM10mm, symbol R
- added C201, C203, C204, C205: 0.1uF, gatedrive:C_Disc, symbol C_Small
- added C202: 330pF, gatedrive:C_Disc, symbol C_Small
- added C206: 100pF, gatedrive:C_Disc, symbol C_Small
- added C207: 10nF, gatedrive:C_Disc, symbol C_Small
- added D201: RGPO2-20, Diodes_ThroughHole:Diode_DO-41_SOD81_Horizontal_RM10, symbol D
- added D202: ~, Diodes_ThroughHole:Diode_DO-201AD_Horizontal_RM15, symbol D
- added IC201: HCPL-316J, Housings_SOIC:SOIC-16_7.5x10.3mm_Pitch1.27mm, symbol HCPL-316J
- added IC202: IXDD614PI, gatedrive:DIP-8_W7.62mm_LongPads, symbol IXDD614PI
- added P201, P202: CONN_01X03, gatedrive:conn, symbol CONN_01X03
- added R201: 10K, Resistors_ThroughHole:Resistor_Horizontal_RM10mm, symbol R_Small
- added R202: 25K, Resistors_ThroughHole:Resistor_Horizontal_RM10mm, symbol R_Small
- added R203, R204: 100, Resistors_ThroughHole:Resistor_Horizontal_RM10mm, symbol R_Small
- added R205: 60, gatedrive:Resistor_multi, symbol R_Small
- added R206: 30ohm ,0.5W, gatedrive:Resistor_multi, symbol R_Small
Connections:
- net 15V7: now also C204.2, C205.1, IC201.12 (Vc), IC201.13 (Vcc2), IC202.1 (VCC), IC202.3 (EN), IC202.8 (VCC), P201.2 (P2)
- net COM7: now also C203.2, C204.1, C206.2, IC201.16 (VE), P201.1 (P1), P202.3 (P3)
- net G7: now also P202.1 (P1), R205.2, R206.2
- net T7: now also IC201.1 (Vin+)
- net c7: now also D201.1 (K), P202.2 (P2)
- net ~FAULT: now also C202.1, IC201.6 (~FAULT), R201.1
- net ~RST: now also IC201.5 (~RESET)
- new net: IC201.11 (Vout), R202.2, R204.2
- new net: C206.1, IC201.14 (DESAT), R203.1
- new net: C207.1, IC202.2 (IN), R204.1
- new net: D201.2 (A), R203.2
- new net: D202.1 (K), R205.1
- new net: D202.2 (A), IC202.6 (OUT), IC202.7 (OUT), R206.1
- new net +5V: C201.1, IC201.3 (Vcc1), R201.2
- new net -5v7: C203.1, C205.2, C207.2, IC201.10 (VEE), IC201.9 (VEE), IC202.4 (GND), IC202.5 (GND), P201.3 (P3), R202.1
- new net GND: C201.2, C202.2, IC201.2 (Vin-), IC201.4 (GND1), IC201.8 (Vled1-)
Other:
- note added: "5 volt is the vcc of the microcontroller.\n"
- note added: "GND is the ground of the microcontroller.\n"
- note added: "IN PIN IS LEFT OPEN OR CONNECTED TO THE VCC."
- note added: "a cap to ensure soft turn-off,\n recommended by datasheet of hcpl."
- note removed: "Fault pull-up resistor."
- note removed: "GND1 is the ground of the microcontroller.\n"
- note removed: "I'M USING GLOBAL LABELS INSTEAD OF LOCAL LABELS AS THEY LOOK NEATER, LOL."
- note removed: "LEFT OPEN OR CONNECTED TO THE VCC."
- note removed: "MICSUPP is 5 volt from the vcc of the microcontroller.\n"
- note removed: "a cap to ensure soft turn-off, recommended by datasheet of hcpl."

Commit message: parting the protection from the GD
Connections:
- net 15V7: now also P201.1 (P1); no longer P201.2 (P2)
- net COM7: now also P201.2 (P2); no longer P201.1 (P1)
Changed lines of the file:
@@
 IN PIN IS LEFT OPEN OR CONNECTED TO THE VCC.
 $Comp
-L PWR_FLAG #FLG09
+L PWR_FLAG #FLG5
 U 1 1 57600D07
 P 1300 3800
-F 0 "#FLG09" H 1300 3895 50  0001 C CNN
+F 0 "#FLG5" H 1300 3895 50  0001 C CNN
 F 1 "PWR_FLAG" H 1300 4024 50  0000 C CNN
 F 2 "" H 1300 3800 50  0000 C CNN
@@
 $EndComp
 $Comp
-L PWR_FLAG #FLG010
+L PWR_FLAG #FLG6
 U 1 1 57600D08
 P 1750 3800
-F 0 "#FLG010" H 1750 3895 50  0001 C CNN
+F 0 "#FLG6" H 1750 3895 50  0001 C CNN
 F 1 "PWR_FLAG" H 1750 4024 50  0000 C CNN
 F 2 "" H 1750 3800 50  0000 C CNN
@@
 $EndComp
 $Comp
-L PWR_FLAG #FLG011
+L PWR_FLAG #FLG4
 U 1 1 57600D0B
 P 1300 2650
-F 0 "#FLG011" H 1300 2745 50  0001 C CNN
+F 0 "#FLG4" H 1300 2745 50  0001 C CNN
 F 1 "PWR_FLAG" H 1300 2874 50  0000 C CNN
 F 2 "" H 1300 2650 50  0000 C CNN
@@
 $EndComp
 $Comp
-L PWR_FLAG #FLG012
+L PWR_FLAG #FLG3
 U 1 1 57600D0C
 P 900 3800
-F 0 "#FLG012" H 900 3895 50  0001 C CNN
+F 0 "#FLG3" H 900 3895 50  0001 C CNN
 F 1 "PWR_FLAG" H 900 4024 50  0000 C CNN
 F 2 "" H 900 3800 50  0000 C CNN
@@
 	-1   0    0    1
 $EndComp
+Text GLabel 1550 4775 2    60   Input ~ 0
+COM7
 Text GLabel 1550 4875 2    60   Input ~ 0
-COM7
-Text GLabel 1550 4775 2    60   Input ~ 0
 15V7
 Text GLabel 1550 5425 2    60   Input ~ 0
@@
 	3975 4150 4150 4150
 $Comp
-L GND #PWR013
+L GND #PWR12
 U 1 1 57600D15
 P 3650 4775
-F 0 "#PWR013" H 3650 4525 50  0001 C CNN
+F 0 "#PWR12" H 3650 4525 50  0001 C CNN
 F 1 "GND" H 3655 4602 50  0000 C CNN
 F 2 "" H 3650 4775 50  0000 C CNN
@@
 	4050 4050 4150 4050
 $Comp
-L +5V #PWR014
+L +5V #PWR11
 U 1 1 57600D16
 P 3650 3650
-F 0 "#PWR014" H 3650 3500 50  0001 C CNN
+F 0 "#PWR11" H 3650 3500 50  0001 C CNN
 F 1 "+5V" H 3665 3823 50  0000 C CNN
 F 2 "" H 3650 3650 50  0000 C CNN
