File: gatedrive.sch (KiCad schematic (older format))
At the start: 7 parts, among them P1 Mic General Connector

Commit message: packup
Parts:
- renumbered D17 to D101, D18 to D102, D19 to D103, P1 to P101, R49 to R101, R50 to R102, R51 to R103
Connections:
- net T2: now also P101.9 (P9); no longer P101.4 (P4)
- net T3: now also P101.8 (P8); no longer P101.5 (P5)
- net T4: now also P101.7 (P7); no longer P101.6 (P6)
- net T5: now also P101.6 (P6); no longer P101.7 (P7)
- net T6: now also P101.5 (P5); no longer P101.8 (P8)
- net T7: now also P101.4 (P4); no longer P101.9 (P9)
- net GND1 renamed GND
- net MICSUPP renamed +5V
- net T8 renamed T1
Changed lines of the file:
@@
 EESchema Schematic File Version 2
+LIBS:gatedrive-rescue
 LIBS:Symbols_DCDC-ACDC-Converter_RevC_20Jul2012
 LIBS:Symbols_EN60617_13Mar2013
@@
 14 Amp IGBT GATE DRIVER CIRCUIT BASED ON  IXDD614PI AND HCPL-316J.
 $Sheet
-S 6650 3950 1650 1300
+S 6425 3875 1650 1300
 U 56EF0567
 F0 "GD7" 60
 F1 "GD7.sch" 60
-F2 "T7" I L 6650 4200 60
-$EndSheet
-$Comp
-L CONN_01X12 P1
+F2 "T7" I L 6425 4125 60
+$EndSheet
+$Comp
+L CONN_01X12 P101
 U 1 1 56EF0F9E
 P 1000 6600
-F 0 "P1" V 1100 6600 50  0000 C CNN
+F 0 "P101" V 1100 6600 50  0000 C CNN
 F 1 "Mic General Connector" V 1200 6625 50  0000 C CNN
 F 2 "Socket_Strips:Socket_Strip_Angled_1x12" H 1000 6600 50  0001 C CNN
@@
 $EndComp
 $Sheet
-S 4000 3950 1650 1300
+S 3775 3875 1650 1300
 U 56EF0565
 F0 "GD6" 60
 F1 "GD6.sch" 60
-F2 "T6" I L 4000 4200 60
-$EndSheet
-$Sheet
-S 1350 3950 1650 1300
+F2 "T6" I L 3775 4125 60
+$EndSheet
+$Sheet
+S 1125 3875 1650 1300
 U 56EF0563
 F0 "GD5" 60
 F1 "GD5.sch" 60
-F2 "T5" I L 1350 4200 60
-$EndSheet
-$Sheet
-S 9300 2050 1650 1300
+F2 "T5" I L 1125 4125 60
+$EndSheet
+$Sheet
+S 9075 1975 1650 1300
 U 56EF0560
 F0 "GD4" 60
 F1 "GD4.sch" 60
-F2 "T4" I L 9300 2200 60
-$EndSheet
-$Sheet
-S 6650 2025 1650 1300
+F2 "T4" I L 9075 2125 60
+$EndSheet
+$Sheet
+S 6425 1950 1650 1300
 U 56EF055E
 F0 "GD3" 60
 F1 "GD3.sch" 60
-F2 "T3" I L 6650 2175 60
-$EndSheet
-$Sheet
-S 4000 2025 1650 1300
+F2 "T3" I L 6425 2100 60
+$EndSheet
+$Sheet
+S 3775 1950 1650 1300
 U 56EF055C
 F0 "GD2" 60
 F1 "GD2.sch" 60
-F2 "T2" I L 4000 2175 60
-$EndSheet
-Text Label 4000 2175 2    60   ~ 0
+F2 "T2" I L 3775 2100 60
+$EndSheet
+Text Label 3775 2100 2    60   ~ 0
 T2
-Text Label 6650 2175 2    60   ~ 0
+Text Label 6425 2100 2    60   ~ 0
 T3
-Text Label 9300 2200 2    60   ~ 0
+Text Label 9075 2125 2    60   ~ 0
 T4
+Text Label 1200 6350 0    60   ~ 0
+T2
+Text Label 1200 6450 0    60   ~ 0
+T3
+Text Label 1200 6550 0    60   ~ 0
+T4
+Text Label 1200 6650 0    60   ~ 0
+T5
+Text Label 1200 6750 0    60   ~ 0
+T6
 Text Label 1200 6850 0    60   ~ 0
-T2
-Text Label 1200 6750 0    60   ~ 0
-T3
-Text Label 1200 6650 0    60   ~ 0
-T4
-Text Label 1200 6550 0    60   ~ 0
-T5
-Text Label 1200 6450 0    60   ~ 0
-T6
-Text Label 1200 6350 0    60   ~ 0
 T7
 Text Label 1200 6250 0    60   ~ 0
-T8
-Text Label 1350 4200 2    60   ~ 0
+T1
+Text Label 1125 4125 2    60   ~ 0
 T5
-Text Label 4000 4200 2    60   ~ 0
+Text Label 3775 4125 2    60   ~ 0
 T6
-Text Label 6650 4200 2    60   ~ 0
+Text Label 6425 4125 2    60   ~ 0
 T7
 Text GLabel 1200 6050 2    60   Input ~ 0
@@
 Text GLabel 1450 6200 3    60   Input ~ 0
 ~RST
-Text GLabel 1200 7050 2    60   Input ~ 0
-GND1
-Text GLabel 1350 7250 3    60   Input ~ 0
-MICSUPP
-Wire Wire Line
-	1350 7250 1350 7150
-Wire Wire Line
-	1350 7150 1200 7150
-$Comp
-L LED D19
+$Comp
+L LED D103
 U 1 1 56F4E3CD
 P 2625 6450
-F 0 "D19" H 2625 6150 50  0000 C CNN
-F 1 "LED" H 2625 6250 50  0000 C CNN
+F 0 "D103" H 2625 6205 50  0000 C CNN
+F 1 "LED" H 2625 6296 50  0000 C CNN
 F 2 "LEDs:LED-3MM" H 2625 6450 50  0001 C CNN
 F 3 "" H 2625 6450 50  0000 C CNN
@@
 $EndComp
 $Comp
-L LED D17
+L LED D101
 U 1 1 56F4E65F
 P 2600 6900
-F 0 "D17" H 2600 6600 50  0000 C CNN
-F 1 "LED" H 2600 6700 50  0000 C CNN
+F 0 "D101" H 2600 6655 50  0000 C CNN
+F 1 "LED" H 2600 6746 50  0000 C CNN
 F 2 "LEDs:LED-3MM" H 2600 6900 50  0001 C CNN
 F 3 "" H 2600 6900 50  0000 C CNN
@@
 $EndComp
 $Comp
-L LED D18
+L LED D102
 U 1 1 56F4E764
 P 2600 7200
-F 0 "D18" H 2600 6900 50  0000 C CNN
-F 1 "LED" H 2600 7000 50  0000 C CNN
+F 0 "D102" H 2600 7350 50  0000 C CNN
+F 1 "LED" H 2600 7450 50  0000 C CNN
 F 2 "LEDs:LED-3MM" H 2600 7200 50  0001 C CNN
 F 3 "" H 2600 7200 50  0000 C CNN
@@
 	-1   0    0    1
 $EndComp
-Text GLabel 3125 6450 2    60   Input ~ 0
-GND1
-Text GLabel 2425 6450 0    60   Input ~ 0
-MICSUPP
-$Comp
-L R R51
+$Comp
+L R R103
 U 1 1 56F4EED0
 P 2975 6450
-F 0 "R51" V 2750 6450 50  0000 C CNN
-F 1 "R" V 2850 6450 50  0000 C CNN
+F 0 "R103" V 2768 6450 50  0000 C CNN
+F 1 "R" V 2859 6450 50  0000 C CNN
 F 2 "Resistors_SMD:R_1206" V 2905 6450 50  0001 C CNN
 F 3 "" H 2975 6450 50  0000 C CNN
@@
 Text GLabel 2400 6900 0    60   Input ~ 0
 ~FAULT
-Text GLabel 3100 6900 2    60   Input ~ 0
-GND1
-$Comp
-L R R49
+$Comp
+L R R101
 U 1 1 56F4F5F2
 P 2950 6900
-F 0 "R49" V 2725 6900 50  0000 C CNN
-F 1 "R" V 2825 6900 50  0000 C CNN
+F 0 "R101" V 2743 6900 50  0000 C CNN
+F 1 "R" V 2834 6900 50  0000 C CNN
 F 2 "Resistors_SMD:R_1206" V 2880 6900 50  0001 C CNN
 F 3 "" H 2950 6900 50  0000 C CNN
@@
 ~RST
 $Comp
-L R R50
+L R R102
 U 1 1 56F4F84D
 P 2950 7200
-F 0 "R50" V 2725 7200 50  0000 C CNN
-F 1 "R" V 2825 7200 50  0000 C CNN
+F 0 "R102" V 2743 7200 50  0000 C CNN
+F 1 "R" V 2834 7200 50  0000 C CNN
 F 2 "Resistors_SMD:R_1206" V 2880 7200 50  0001 C CNN
 F 3 "" H 2950 7200 50  0000 C CNN
@@
 	0    1    1    0
 $EndComp
-Text GLabel 3100 7200 2    60   Input ~ 0
-GND1
 Wire Notes Line
 	1800 6075 3650 6075
@@
 	725  7675 725  5800
 $Sheet
-S 9300 3950 1650 1300
+S 9075 3875 1650 1300
 U 56FD530B
-F0 "Sheet56FD530A" 60
+F0 "protection" 60
 F1 "Protection.sch" 60
 $EndSheet
@@
 Text Notes 4750 950  0    60   ~ 0
 the circuit  drives 8 IGBTs  suitable for inverter and motor control applications.
-Text Label 1350 2300 2    60   ~ 0
-T8
-$Sheet
-S 1350 2050 1650 1300
+Text Label 1125 2225 2    60   ~ 0
+T1
+$Sheet
+S 1125 1975 1650 1300
 U 56EF0569
-F0 "GD8" 60
-F1 "GD8.sch" 60
-F2 "T8" I L 1350 2300 60
+F0 "GD1" 60
+F1 "GD1.sch" 60
+F2 "T1" I L 1125 2225 60
 $EndSheet
 Text GLabel 1450 6950 1    60   Input ~ 0
@@
 Wire Wire Line
 	1450 6950 1200 6950
+$Comp
+L GND #PWR01
+U 1 1 576064B1
+P 1525 7250
+F 0 "#PWR01" H 1525 7000 50  0001 C CNN
+F 1 "GND" H 1530 7077 50  0000 C CNN
+F 2 "" H 1525 7250 50  0000 C CNN
+F 3 "" H 1525 7250 50  0000 C CNN
+	1    1525 7250
+	1    0    0    -1
+$EndComp
+$Comp
+L +5V #PWR02
+U 1 1 57606519
+P 2425 6450
+F 0 "#PWR02" H 2425 6300 50  0001 C CNN
+F 1 "+5V" V 2440 6578 50  0000 L CNN
+F 2 "" H 2425 6450 50  0000 C CNN
+F 3 "" H 2425 6450 50  0000 C CNN
+	1    2425 6450
+	0    -1   -1   0
+$EndComp
+Wire Wire Line
+	1525 7250 1525 7050
+Wire Wire Line
+	1525 7050 1200 7050
+$Comp
+L GND #PWR03
+U 1 1 57606699
+P 3300 6800
+F 0 "#PWR03" H 3300 6550 50  0001 C CNN
+F 1 "GND" V 3305 6672 50  0000 R CNN
+F 2 "" H 3300 6800 50  0000 C CNN
+F 3 "" H 3300 6800 50  0000 C CNN
+	1    3300 6800
+	0    -1   -1   0
+$EndComp
+Wire Wire Line
+	3125 6450 3225 6450
+Wire Wire Line
+	3225 6450 3225 7200
+Wire Wire Line
+	3225 6800 3300 6800
+Wire Wire Line
+	3225 7200 3100 7200
+Connection ~ 3225 6800
+Wire Wire Line
+	3100 6900 3225 6900
+Connection ~ 3225 6900
+$Comp
+L +5V #PWR04
+U 1 1 5760A969
+P 1350 7250
+F 0 "#PWR04" H 1350 7100 50  0001 C CNN
+F 1 "+5V" V 1365 7378 50  0000 L CNN
+F 2 "" H 1350 7250 50  0000 C CNN
+F 3 "" H 1350 7250 50  0000 C CNN
+	1    1350 7250
+	-1   0    0    1
+$EndComp
+Wire Wire Line
+	1350 7250 1350 7150
+Wire Wire Line
+	1350 7150 1200 7150
+$Comp
+L +5V #PWR05
+U 1 1 576D9A68
+P 3950 6375
+F 0 "#PWR05" H 3950 6225 50  0001 C CNN
+F 1 "+5V" V 3965 6503 50  0000 L CNN
+F 2 "" H 3950 6375 50  0000 C CNN
+F 3 "" H 3950 6375 50  0000 C CNN
+	1    3950 6375
+	1    0    0    -1
+$EndComp
+$Comp
+L GND #PWR06
+U 1 1 576D9ADC
+P 3950 6600
+F 0 "#PWR06" H 3950 6350 50  0001 C CNN
+F 1 "GND" V 3955 6472 50  0000 R CNN
+F 2 "" H 3950 6600 50  0000 C CNN
+F 3 "" H 3950 6600 50  0000 C CNN
+	1    3950 6600
+	1    0    0    -1
+$EndComp
+$Comp
+L PWR_FLAG #FLG07
+U 1 1 576D9BAD
+P 3950 6375
+F 0 "#FLG07" H 3950 6470 50  0001 C CNN
+F 1 "PWR_FLAG" V 3950 6553 50  0000 L CNN
+F 2 "" H 3950 6375 50  0000 C CNN
+F 3 "" H 3950 6375 50  0000 C CNN
+	1    3950 6375
+	0    1    1    0
+$EndComp
+$Comp
+L PWR_FLAG #FLG08
+U 1 1 576D9C1A
+P 3950 6600
+F 0 "#FLG08" H 3950 6695 50  0001 C CNN
+F 1 "PWR_FLAG" V 3950 6778 50  0000 L CNN
+F 2 "" H 3950 6600 50  0000 C CNN
+F 3 "" H 3950 6600 50  0000 C CNN
+	1    3950 6600
+	0    1    1    0
+$EndComp
 $EndSCHEMATC

Commit message: parting the protection from the GD
Parts:
- added P1, P2: CONN_01X03, Pin_Headers:Pin_Header_Angled_1x04, symbol CONN_01X04
- P101: footprint Socket_Strips:Socket_Strip_Angled_1x12 -> gatedrive:MICCONN
Connections:
- net +5V: now also P1.3 (P3), P2.2 (P2)
- net GND: now also P1.1 (P1), P2.4 (P4)
- net ~FAULT: now also P1.4 (P4), P2.1 (P1)
- net ~OVERTEMP: now also P1.2 (P2), P2.3 (P3)
Changed lines of the file:
@@
 F 0 "P101" V 1100 6600 50  0000 C CNN
 F 1 "Mic General Connector" V 1200 6625 50  0000 C CNN
-F 2 "Socket_Strips:Socket_Strip_Angled_1x12" H 1000 6600 50  0001 C CNN
+F 2 "gatedrive:MICCONN" H 1000 6600 50  0001 C CNN
 F 3 "" H 1000 6600 50  0000 C CNN
 	1    1000 6600
@@
 	1450 6950 1200 6950
 $Comp
-L GND #PWR01
+L GND #PWR2
 U 1 1 576064B1
 P 1525 7250
-F 0 "#PWR01" H 1525 7000 50  0001 C CNN
+F 0 "#PWR2" H 1525 7000 50  0001 C CNN
 F 1 "GND" H 1530 7077 50  0000 C CNN
 F 2 "" H 1525 7250 50  0000 C CNN
@@
 $EndComp
 $Comp
-L +5V #PWR02
+L +5V #PWR3
 U 1 1 57606519
 P 2425 6450
-F 0 "#PWR02" H 2425 6300 50  0001 C CNN
+F 0 "#PWR3" H 2425 6300 50  0001 C CNN
 F 1 "+5V" V 2440 6578 50  0000 L CNN
 F 2 "" H 2425 6450 50  0000 C CNN
@@
 	1525 7050 1200 7050
 $Comp
-L GND #PWR03
+L GND #PWR4
 U 1 1 57606699
 P 3300 6800
-F 0 "#PWR03" H 3300 6550 50  0001 C CNN
+F 0 "#PWR4" H 3300 6550 50  0001 C CNN
 F 1 "GND" V 3305 6672 50  0000 R CNN
 F 2 "" H 3300 6800 50  0000 C CNN
@@
 Connection ~ 3225 6900
 $Comp
-L +5V #PWR04
+L +5V #PWR1
 U 1 1 5760A969
 P 1350 7250
-F 0 "#PWR04" H 1350 7100 50  0001 C CNN
+F 0 "#PWR1" H 1350 7100 50  0001 C CNN
 F 1 "+5V" V 1365 7378 50  0000 L CNN
 F 2 "" H 1350 7250 50  0000 C CNN
@@
 	1350 7150 1200 7150
 $Comp
-L +5V #PWR05
+L +5V #PWR5
 U 1 1 576D9A68
 P 3950 6375
-F 0 "#PWR05" H 3950 6225 50  0001 C CNN
+F 0 "#PWR5" H 3950 6225 50  0001 C CNN
 F 1 "+5V" V 3965 6503 50  0000 L CNN
 F 2 "" H 3950 6375 50  0000 C CNN
@@
 $EndComp
 $Comp
-L GND #PWR06
+L GND #PWR6
 U 1 1 576D9ADC
 P 3950 6600
-F 0 "#PWR06" H 3950 6350 50  0001 C CNN
+F 0 "#PWR6" H 3950 6350 50  0001 C CNN
 F 1 "GND" V 3955 6472 50  0000 R CNN
 F 2 "" H 3950 6600 50  0000 C CNN
@@
 $EndComp
 $Comp
-L PWR_FLAG #FLG07
+L PWR_FLAG #FLG1
 U 1 1 576D9BAD
 P 3950 6375
-F 0 "#FLG07" H 3950 6470 50  0001 C CNN
+F 0 "#FLG1" H 3950 6470 50  0001 C CNN
 F 1 "PWR_FLAG" V 3950 6553 50  0000 L CNN
 F 2 "" H 3950 6375 50  0000 C CNN
@@
 $EndComp
 $Comp
-L PWR_FLAG #FLG08
+L PWR_FLAG #FLG2
 U 1 1 576D9C1A
 P 3950 6600
-F 0 "#FLG08" H 3950 6695 50  0001 C CNN
+F 0 "#FLG2" H 3950 6695 50  0001 C CNN
 F 1 "PWR_FLAG" V 3950 6778 50  0000 L CNN
 F 2 "" H 3950 6600 50  0000 C CNN
@@
 	0    1    1    0
 $EndComp
+$Comp
+L CONN_01X04 P1
+U 1 1 5773A312
+P 4925 6275
+F 0 "P1" H 4844 5900 50  0000 C CNN
+F 1 "CONN_01X03" H 4844 5991 50  0000 C CNN
+F 2 "Pin_Headers:Pin_Header_Angled_1x04" H 4844 5992 50  0001 C CNN
+F 3 "" H 4925 6275 50  0000 C CNN
+	1    4925 6275
+	-1   0    0    1
+$EndComp
+$Comp
+L GND #PWR7
+U 1 1 5773A441
+P 5125 6425
+F 0 "#PWR7" H 5125 6175 50  0001 C CNN
+F 1 "GND" V 5130 6297 50  0000 R CNN
+F 2 "" H 5125 6425 50  0000 C CNN
+F 3 "" H 5125 6425 50  0000 C CNN
+	1    5125 6425
+	1    0    0    -1
+$EndComp
+$Comp
+L +5V #PWR8
+U 1 1 5773A48E
+P 5500 6175
+F 0 "#PWR8" H 5500 6025 50  0001 C CNN
+F 1 "+5V" V 5515 6303 50  0000 L CNN
+F 2 "" H 5500 6175 50  0000 C CNN
+F 3 "" H 5500 6175 50  0000 C CNN
+	1    5500 6175
+	1    0    0    -1
+$EndComp
+Text GLabel 5275 6400 3    60   Input ~ 0
+~OVERTEMP
+Text GLabel 5125 6125 2    60   Input ~ 0
+~FAULT
+Wire Wire Line
+	5275 6400 5275 6325
+Wire Wire Line
+	5275 6325 5125 6325
+Wire Wire Line
+	5125 6225 5500 6225
+Wire Wire Line
+	5500 6225 5500 6175
+$Comp
+L CONN_01X04 P2
+U 1 1 57745AD3
+P 6650 6325
+F 0 "P2" H 6568 6690 50  0000 C CNN
+F 1 "CONN_01X03" H 6568 6599 50  0000 C CNN
+F 2 "Pin_Headers:Pin_Header_Angled_1x04" H 6569 6042 50  0001 C CNN
+F 3 "" H 6650 6325 50  0000 C CNN
+	1    6650 6325
+	1    0    0    -1
+$EndComp
+$Comp
+L GND #PWR9
+U 1 1 57745AD9
+P 6450 6475
+F 0 "#PWR9" H 6450 6225 50  0001 C CNN
+F 1 "GND" V 6455 6347 50  0000 R CNN
+F 2 "" H 6450 6475 50  0000 C CNN
+F 3 "" H 6450 6475 50  0000 C CNN
+	1    6450 6475
+	1    0    0    -1
+$EndComp
+$Comp
+L +5V #PWR10
+U 1 1 57745ADF
+P 6075 6250
+F 0 "#PWR10" H 6075 6100 50  0001 C CNN
+F 1 "+5V" V 6090 6378 50  0000 L CNN
+F 2 "" H 6075 6250 50  0000 C CNN
+F 3 "" H 6075 6250 50  0000 C CNN
+	1    6075 6250
+	1    0    0    -1
+$EndComp
+Text GLabel 6275 6475 3    60   Input ~ 0
+~OVERTEMP
+Text GLabel 6450 6175 0    60   Input ~ 0
+~FAULT
+Wire Wire Line
+	6075 6250 6075 6275
+Wire Wire Line
+	6075 6275 6450 6275
+Wire Wire Line
+	6275 6475 6275 6375
+Wire Wire Line
+	6275 6375 6450 6375
 $EndSCHEMATC
